File: KKK_valdiklis1.brd (EAGLE design)
At the start: 160 x 100 mm, 71 parts, among them IC1 MCP1702-3.3, IC2 L293D, IC3 MCP1702-5.0, IC4 ATMEGA1284, IC5 DS1307, K1 S202T02, K2 S202T02, K3 S202T02, K4 S202T02, K5 S202T02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

Commit message: projektavimas
Parts:
- removed K6: S202T02, relay-1:S202T02
- removed X2: Storage tank pump, con-molex:22-23-2021
- removed X3: Radiator pump, con-molex:22-23-2021
- removed X5: 4 way valve 2, con-molex:22-23-2021
- removed X6: Floor heating, con-molex:22-23-2021
- removed X77: PUMP1, con-molex:22-23-2041
- removed X88: PUMP2, con-molex:22-23-2041
- added K7: S202T02, relay-1:S202T02
- X1: value Boiler pump -> PUMP; device con-molex:22-23-2021 -> con-molex:22-23-2041
- X4: value 4 way valve 1 -> PUMP; device con-molex:22-23-2021 -> con-molex:22-23-2041
- moved R15 237.2 mm to (144.8, -15.2), turned to 90 degrees
- moved D4 215.8 mm to (99.1, -15.2), turned to 90 degrees
- moved R14 213.7 mm to (138.4, -1.27), turned to 90 degrees
- moved IC2 213.3 mm to (-29.8, -102.2)
- moved X10 211.4 mm to (130.2, 19.1)
- moved R17 203.0 mm to (-18.4, -93.3), turned to 180 degrees
- moved R12 200.3 mm to (55.9, -15.2), turned to 90 degrees
- moved Q4 196.8 mm to (133.3, -5.08), turned to 90 degrees
- moved BAT1 196.3 mm to (96.5, 53.3), turned to 180 degrees
- moved R16 190.5 mm to (-19.1, -81.3), turned to 180 degrees
- moved R7 190.4 mm to (-19.1, -69.2), turned to 180 degrees
- moved IC5 186.5 mm to (128.3, -14.0), turned to 90 degrees
- moved R13 181.5 mm to (104.1, -15.2), turned to 90 degrees
- moved R4 172.3 mm to (-19.1, -59.7), turned to 180 degrees
- moved C8 171.8 mm to (48.3, 25.1), turned to 180 degrees
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Connections:
- net +12V renamed VCC2
- removed net D6: IC2.2
- removed net D7: IC2.7
- removed net D8: IC2.15
- removed net D9: IC2.10
- removed net MV1.1: IC2.3
- removed net MV1.2: IC2.6
- removed net MV2.1: IC2.14
- removed net MV2.2: IC2.11
- new net D5(MOSI): IC4.6
- new net GND2: IC2.5
- new net GND3: IC2.13
- new net GND4: IC2.12
- new net VCC1: IC2.16
- net +5V: no longer IC2.16
- net D5: no longer IC4.6
- net GND: now also K7.K, X4.3, X4.4; no longer IC2.12, IC2.13, IC2.4, IC2.5, K6.K, X77.3, X77.4
- net GND1: now also IC2.4, X1.3, X1.4; no longer X88.3, X88.4
- net N$15: now also X4.1, X4.2; no longer X77.1, X77.2
- net N$16: now also K1.A; no longer K3.A
- net N$18: now also K1.DS1; no longer K3.DS1, X3.1
- net N$19: now also X1.1, X1.2; no longer X88.1, X88.2
- net N$23: now also K1.DS2; no longer K3.DS2, X3.2
- net N$25: no longer X2.1
- net N$26: no longer X2.2
- net N$28: now also K7.A; no longer K4.A
- net N$29: now also K7.DS1; no longer K4.DS1, X4.1
- net N$30: now also K7.DS2; no longer K4.DS2, X4.2
- net N$31: now also K3.A; no longer K1.A
- net N$32: now also K3.DS1; no longer K1.DS1, X1.1
- net N$33: now also K3.DS2; no longer K1.DS2, X1.2
- net N$34: now also K4.A; no longer K6.A
- net N$35: now also K4.DS1; no longer K6.DS1, X6.1
- net N$36: now also K4.DS2; no longer K6.DS2, X6.2
- net N$38: no longer X5.1
- net N$39: no longer X5.2
Other:
- board size 160 x 100 mm -> 100 x 87 mm
- board text added: "5V"
- board text added: ">DRAWING_NAME"
- board text added: ">PLOT_DATE_TIME"
- board text added: "BLACK"
- board text added: "DTR"
- board text added: "GND"
- board text added: "GREEN"
- board text added: "MHz"
- board text added: "RESET"
