File: KKK_valdiklis.brd (EAGLE design)
At the start: 100 x 87 mm, 72 parts, among them IC1 MCP1702-3.3, IC3 MCP1702-5.0, IC4 ATMEGA1284, IC5 DS1307, K1 S202T02, K2 S202T02, K3 S202T02, K4 S202T02, K5 S202T02, K7 S202T02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

Commit message: eiga...
Parts:
- removed X13, X14, X15, X5, X6, X7, X8, X9: (no value), con-phoenix-254:3POL254
Connections:
- net 11(MOSI) renamed D5(MOSI)
- net 12(MISO) renamed D6(MISO)
- net 14 renamed D23
- net 15 renamed D22
- net 16(TDI) renamed D21
- net 17(TDO) renamed D20(TDO)
- net 18(TMS) renamed D19(TMS)
- net 19(TCK) renamed D18(TCK)
- net 2(RX1) renamed D102(RX1)
- net 22 renamed D12
- net 23 renamed D15
- net 3(TX1) renamed D11(TX1)
- net 4 renamed D0
- net 8 renamed D14
- net 9 renamed D13
- removed net 10: IC4.5
- removed net 5: IC4.2
- removed net 6: IC4.3
- removed net 7: IC4.4
- new net D16(SCL): IC4.22
- new net D17(SDA): IC4.23
- new net D7(SCK): IC4.8
- new net D8(RX0): IC4.14
- new net D9(TX0): IC4.15
- net +5V: no longer X13.3, X14.3, X15.3, X5.3, X6.3, X7.3, X8.3, X9.3
- net 0(RX0): no longer IC4.14
- net 1(TX0): no longer IC4.15
- net 13(SCK): no longer IC4.8
- net 20(SDA): no longer IC4.23
- net 21(SCL): no longer IC4.22
- net A0: now also IC4.40; no longer IC4.33
- net A1: now also IC4.39; no longer IC4.34, X14.2, X6.2, X9.2
- net A2: now also IC4.38; no longer IC4.35
- net A3: now also IC4.37; no longer IC4.36
- net A4: now also IC4.36; no longer IC4.37
- net A5: now also IC4.35; no longer IC4.38
- net A6: now also IC4.34; no longer IC4.39
- net A7: now also IC4.33; no longer IC4.40
- net D1: now also IC4.2; no longer X13.2, X5.2, X8.2
- net D2: now also IC4.3; no longer X15.2, X7.2
- net D3: now also IC4.4
- net D4: now also IC4.5
- net GND: no longer X13.1, X14.1, X15.1, X5.1, X6.1, X7.1, X8.1, X9.1

Commit message: projektavimas
Parts:
- added IC2: L293D, st-microelectronics:DIL16
Connections:
- removed net D6: R4.1
- removed net D7: R7.1
- removed net D8: R16.1
- removed net D9: R17.1
- new net GND2: IC2.5
- new net GND3: IC2.13
- new net GND4: IC2.12
- new net VCC1: IC2.16
- new net VCC2: IC2.8
- net D0: now also R5.1
- net D1: now also R17.1
- net D2: now also R16.1
- net D3: now also R7.1
- net D4: now also R4.1; no longer R3.1
- net D5: now also R3.1; no longer R5.1
- net GND1: now also IC2.4
Changed lines of the file:
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@@
 <element name="K5" library="relay-1" package="S202T02" value="S202T02" x="-33.655" y="-86.995"/>
 <element name="R17" library="resistor-1" package="0207/10" value="330" x="-35.56" y="-94.615"/>
+<element name="IC2" library="st-microelectronics" package="DIL16" value="L293D" x="-29.845" y="-102.235">
+<attribute name="OC_NEWARK" value="56P8249" x="-29.845" y="-102.235" size="1.778" layer="27" display="off"/>
+<attribute name="MPN" value="L293D" x="-29.845" y="-102.235" size="1.778" layer="27" display="off"/>
+<attribute name="MF" value="" x="-29.845" y="-102.235" size="1.778" layer="27" display="off"/>
+<attribute name="OC_FARNELL" value="9589619" x="-29.845" y="-102.235" size="1.778" layer="27" display="off"/>
+</element>
 </elements>
 <signals>
@@
 <signal name="D0">
 <contactref element="IC4" pad="1"/>
+<contactref element="R5" pad="1"/>
+<wire x1="-40.64" y1="-37.465" x2="53.34" y2="59.69" width="0" layer="19" extent="1-1"/>
 </signal>
 <signal name="D1">
 <contactref element="IC4" pad="2"/>
+<contactref element="R17" pad="1"/>
+<wire x1="50.8" y1="59.69" x2="-40.64" y2="-94.615" width="0" layer="19" extent="1-1"/>
 </signal>
 <signal name="D23">
@@
 <contactref element="R13" pad="1"/>
 <contactref element="IC4" pad="4"/>
-<wire x1="55.88" y1="-20.32" x2="45.72" y2="59.69" width="0" layer="19" extent="1-1"/>
+<contactref element="R7" pad="1"/>
+<wire x1="55.88" y1="-20.32" x2="-40.64" y2="-71.755" width="0" layer="19" extent="1-1"/>
 <wire x1="104.14" y1="-20.32" x2="55.88" y2="-20.32" width="0" layer="19" extent="1-1"/>
+<wire x1="45.72" y1="59.69" x2="55.88" y2="-20.32" width="0" layer="19" extent="1-1"/>
 </signal>
 <signal name="N$13">
@@
 <contactref element="X1" pad="3"/>
 <contactref element="X1" pad="4"/>
-<wire x1="88.9" y1="-11.43" x2="99.06" y2="-10.16" width="0" layer="19" extent="1-1"/>
+<contactref element="IC2" pad="4"/>
+<wire x1="77.47" y1="-12.7" x2="-31.115" y2="-106.045" width="0" layer="19" extent="1-1"/>
+<wire x1="88.9" y1="-11.43" x2="77.47" y2="-12.7" width="0" layer="19" extent="1-1"/>
 <wire x1="88.9" y1="-13.97" x2="88.9" y2="-11.43" width="0" layer="19" extent="1-1"/>
-<wire x1="77.47" y1="-12.7" x2="88.9" y2="-11.43" width="0" layer="19" extent="1-1"/>
+<wire x1="99.06" y1="-10.16" x2="88.9" y2="-11.43" width="0" layer="19" extent="1-1"/>
 </signal>
 <signal name="N$17">
@@
 <contactref element="X10" pad="2"/>
 <contactref element="IC4" pad="3"/>
+<contactref element="R16" pad="1"/>
 <wire x1="48.26" y1="59.69" x2="130.175" y2="19.05" width="0" layer="19" extent="1-1"/>
+<wire x1="-40.64" y1="-83.185" x2="48.26" y2="59.69" width="0" layer="19" extent="1-1"/>
 </signal>
 <signal name="N$5">
@@
 <wire x1="132.08" y1="-12.7" x2="76.52" y2="53.34" width="0" layer="19" extent="1-1"/>
 </signal>
-<signal name="D5">
-<contactref element="R5" pad="1"/>
-</signal>
 <signal name="N$28">
 <contactref element="K7" pad="A"/>
@@
 </signal>
 <signal name="D4">
-<contactref element="R3" pad="1"/>
 <contactref element="IC4" pad="5"/>
-<wire x1="-40.64" y1="-48.895" x2="43.18" y2="59.69" width="0" layer="19" extent="1-1"/>
+<contactref element="R4" pad="1"/>
+<wire x1="-40.64" y1="-60.325" x2="43.18" y2="59.69" width="0" layer="19" extent="1-1"/>
 </signal>
 <signal name="N$16">
@@
 <contactref element="K1" pad="DS2"/>
 </signal>
-<signal name="D6">
-<contactref element="R4" pad="1"/>
-</signal>
 <signal name="N$24">
 <contactref element="K2" pad="A"/>
@@
 <contactref element="K2" pad="DS2"/>
 </signal>
-<signal name="D7">
-<contactref element="R7" pad="1"/>
-</signal>
 <signal name="N$31">
 <contactref element="K3" pad="A"/>
@@
 <contactref element="K3" pad="DS2"/>
 </signal>
-<signal name="D8">
-<contactref element="R16" pad="1"/>
-</signal>
 <signal name="N$34">
 <contactref element="K4" pad="A"/>
@@
 <contactref element="K4" pad="DS2"/>
 </signal>
-<signal name="D9">
-<contactref element="R17" pad="1"/>
-</signal>
 <signal name="N$37">
 <contactref element="K5" pad="A"/>
@@
 <contactref element="IC4" pad="8"/>
 </signal>
+<signal name="D5">
+<contactref element="R3" pad="1"/>
+</signal>
+<signal name="GND2">
+<contactref element="IC2" pad="5"/>
+</signal>
+<signal name="VCC2">
+<contactref element="IC2" pad="8"/>
+</signal>
+<signal name="VCC1">
+<contactref element="IC2" pad="16"/>
+</signal>
+<signal name="GND3">
+<contactref element="IC2" pad="13"/>
+</signal>
+<signal name="GND4">
+<contactref element="IC2" pad="12"/>
+</signal>
 </signals>

Commit message: projektavimas
Parts:
- removed K7: S202T02, relay-1:S202T02
- removed LED1: D13, SparkFun:LED3MM
- removed Q1: 2N7000, SteveMarple:TO-92
- removed R1: 1k, SteveMarple:RES-AXIAL-0.4
- removed R10: 1M, SteveMarple:RES-AXIAL-0.4
- added K6: S202T02, relay-1:S202T02
- added X2: Storage tank pump, con-molex:22-23-2021
- added X3: Radiator pump, con-molex:22-23-2021
- added X5: 4 way valve 2, con-molex:22-23-2021
- added X6: Floor heating, con-molex:22-23-2021
- added X77: PUMP1, con-molex:22-23-2041
- added X88: PUMP2, con-molex:22-23-2041
- X1: value PUMP -> Boiler pump; device con-molex:22-23-2041 -> con-molex:22-23-2021
- X4: value PUMP -> 4 way valve 1; device con-molex:22-23-2041 -> con-molex:22-23-2021
- moved R15 237.2 mm to (-57.1, 109.2), turned to 0 degrees
- moved D4 215.8 mm to (-92.7, 83.8), turned to 0 degrees
- moved R14 213.7 mm to (-44.5, 109.2), turned to 0 degrees
- moved IC2 213.3 mm to (137.2, 30.5)
- moved X10 211.4 mm to (-66.0, 97.8)
- moved R17 203.9 mm to (-31.8, 109.2)
- moved R12 200.3 mm to (-99.1, 111.8), turned to 0 degrees
- moved Q4 196.8 mm to (-53.3, 57.1), turned to 0 degrees
- moved BAT1 196.3 mm to (-95.2, 11.4), turned to 0 degrees
- moved R16 193.1 mm to (-19.1, 109.2)
- moved R7 186.6 mm to (-97.8, 104.1)
- moved IC5 186.5 mm to (-41.9, 62.2), turned to 0 degrees
- moved R13 181.5 mm to (-20.3, 116.8), turned to 0 degrees
- moved C8 171.8 mm to (-97.8, 115.6), turned to 0 degrees
- moved R4 168.5 mm to (-72.4, 104.1)
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Connections:
- net VCC2 renamed +12V
- removed net 13(SCK): Q1.2, R10.P$2
- removed net 20(SDA): IC5.5, R15.1
- removed net 21(SCL): IC5.6, R14.2
- removed net D5(MOSI): IC4.6
- removed net GND2: IC2.5
- removed net GND3: IC2.13
- removed net GND4: IC2.12
- removed net N$3: LED1.A, R1.P$1
- removed net N$4: LED1.K, Q1.3
- removed net VCC1: IC2.16
- new net D6: IC2.2, R12.1
- new net D7: IC2.7, R13.1
- new net D8: IC2.15
- new net D9: IC2.10
- new net MV1.1: IC2.3
- new net MV1.2: IC2.6
- new net MV2.1: IC2.14
- new net MV2.2: IC2.11
- net +5V: now also IC2.16
- net D0: now also R7.1; no longer R5.1
- net D1: now also R4.1; no longer R17.1
- net D16(SCL): now also IC5.6, R14.2
- net D17(SDA): now also IC5.5, R15.1
- net D2: now also R3.1; no longer R16.1
- net D3: now also R5.1; no longer R12.1, R13.1, R7.1
- net D4: now also R17.1; no longer R4.1
- net D5: now also IC4.6, R16.1; no longer R3.1
- net GND: now also IC2.12, IC2.13, IC2.4, IC2.5, K6.K, X77.3, X77.4; no longer K7.K, Q1.1, R10.P$1, X4.3, X4.4
- net GND1: now also X88.3, X88.4; no longer IC2.4, X1.3, X1.4
- net N$15: now also X77.1, X77.2; no longer X4.1, X4.2
- net N$16: now also K3.A; no longer K1.A
- net N$18: now also K3.DS1, X3.1; no longer K1.DS1
- net N$19: now also X88.1, X88.2; no longer X1.1, X1.2
- net N$23: now also K3.DS2, X3.2; no longer K1.DS2
- net N$25: now also X2.1
- net N$26: now also X2.2
- net N$28: now also K4.A; no longer K7.A
- net N$29: now also K4.DS1, X4.1; no longer K7.DS1
- net N$30: now also K4.DS2, X4.2; no longer K7.DS2
- net N$31: now also K1.A; no longer K3.A
- net N$32: now also K1.DS1, X1.1; no longer K3.DS1
- net N$33: now also K1.DS2, X1.2; no longer K3.DS2
- net N$34: now also K6.A; no longer K4.A
- net N$35: now also K6.DS1, X6.1; no longer K4.DS1
- net N$36: now also K6.DS2, X6.2; no longer K4.DS2
- net N$38: now also X5.1
- net N$39: now also X5.2
- net VCC: no longer R1.P$2
Other:
- board size 100 x 87 mm -> 160 x 100 mm
- board text removed: "5V"
- board text removed: ">DRAWING_NAME"
- board text removed: ">PLOT_DATE_TIME"
- board text removed: "BLACK"
- board text removed: "DTR"
- board text removed: "GND"
- board text removed: "GREEN"
- board text removed: "MHz"
- board text removed: "RESET"

Commit message: projektavimas
Parts:
- added X7: motorized valve 1, con-molex:22-23-2021
- added X8: motorized valve 2, con-molex:22-23-2021
Connections:
- net MV1.1: now also X7.1
- net MV1.2: now also X7.2
- net MV2.1: now also X8.1
- net MV2.2: now also X8.2
Changed lines of the file:
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@@
 <attribute name="OC_FARNELL" value="1462926" x="123.19" y="-72.39" size="1.778" layer="27" display="off"/>
+</element>
+<element name="X7" library="con-molex" package="22-23-2021" value="motorized valve 1" x="-115.57" y="-6.35">
+<attribute name="OC_NEWARK" value="25C3832" x="-115.57" y="-6.35" size="1.778" layer="27" display="off"/>
+<attribute name="MPN" value="22-23-2021" x="-115.57" y="-6.35" size="1.778" layer="27" display="off"/>
+<attribute name="MF" value="MOLEX" x="-115.57" y="-6.35" size="1.778" layer="27" display="off"/>
+<attribute name="OC_FARNELL" value="1462926" x="-115.57" y="-6.35" size="1.778" layer="27" display="off"/>
+</element>
+<element name="X8" library="con-molex" package="22-23-2021" value="motorized valve 2" x="-123.19" y="-6.35">
+<attribute name="OC_NEWARK" value="25C3832" x="-123.19" y="-6.35" size="1.778" layer="27" display="off"/>
+<attribute name="MPN" value="22-23-2021" x="-123.19" y="-6.35" size="1.778" layer="27" display="off"/>
+<attribute name="MF" value="MOLEX" x="-123.19" y="-6.35" size="1.778" layer="27" display="off"/>
+<attribute name="OC_FARNELL" value="1462926" x="-123.19" y="-6.35" size="1.778" layer="27" display="off"/>
 </element>
 </elements>
@@
 <signal name="MV1.1">
 <contactref element="IC2" pad="3"/>
+<contactref element="X7" pad="1"/>
+<wire x1="-116.84" y1="-6.35" x2="133.35" y2="26.67" width="0" layer="19" extent="1-1"/>
 </signal>
 <signal name="MV1.2">
 <contactref element="IC2" pad="6"/>
+<contactref element="X7" pad="2"/>
+<wire x1="-114.3" y1="-6.35" x2="140.97" y2="26.67" width="0" layer="19" extent="1-1"/>
 </signal>
 <signal name="D7">
@@
 <signal name="MV2.1">
 <contactref element="IC2" pad="14"/>
+<contactref element="X8" pad="1"/>
+<wire x1="-124.46" y1="-6.35" x2="133.35" y2="34.29" width="0" layer="19" extent="1-1"/>
 </signal>
 <signal name="MV2.2">
 <contactref element="IC2" pad="11"/>
+<contactref element="X8" pad="2"/>
+<wire x1="-121.92" y1="-6.35" x2="140.97" y2="34.29" width="0" layer="19" extent="1-1"/>
 </signal>
 <signal name="D9">

Commit message: projektavimas
Parts:
- removed D4: 1N4004, diode:DO41-10
- removed Q3: TIP120V, rocketfarm:TO220AV
- removed R13: 2k, resistor:0207/10
- removed X88: PUMP2, con-molex:22-23-2041
- C17: device rcl:C0805K -> rcl:C025-024X044
- moved S2 254.7 mm to (156.2, 91.4)
- moved BAT1 234.6 mm to (134.6, 58.4)
- moved X7 221.2 mm to (105.4, 2.54), turned to 180 degrees
- moved X8 219.9 mm to (96.5, 2.54), turned to 180 degrees
- moved R9 215.3 mm to (152.4, 80.0)
- moved D3 212.5 mm to (121.9, 17.8)
- moved R8 186.3 mm to (135.9, 81.3)
- moved R11 185.8 mm to (148.6, 83.8)
- moved Q4 175.3 mm to (121.9, 58.4), turned to 180 degrees
- moved S4 172.8 mm to (142.2, 90.2)
- moved IC5 166.4 mm to (124.5, 66.0)
- moved S1 152.4 mm to (64.8, 72.4)
- moved S3 143.7 mm to (124.5, 91.4)
- moved C3 126.1 mm to (14.0, 74.9)
- moved Y1 110.8 mm to (12.7, 63.5)
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Connections:
- removed net GND1: D4.A, Q3.E, X88.3, X88.4
- removed net N$17: Q3.B, R13.2
- removed net N$19: D4.C, Q3.C, X88.1, X88.2
- new net D10: U$1.P$11
- new net D11: U$1.P$10
- net +3V3: now also U$1.P$16
- net D12: now also U$1.P$9
- net D13: now also U$1.P$12
- net D14: now also U$1.P$13
- net D15: now also U$1.P$14
- net D7: no longer R13.1
- net GND: now also U$1.P$15, X77.1, X77.2; no longer X77.3, X77.4
- net N$15: now also X77.3, X77.4; no longer X77.1, X77.2
