File: KKK_valdiklis.brd (EAGLE design)
At the start: 160 x 100 mm, 65 parts, among them IC1 MCP1702-3.3, IC2 L293D, IC3 MCP1702-5.0, IC4 ATMEGA1284, IC5 DS1307, K1 S202T02, K2 S202T02, K3 S202T02, K4 S202T02, K5 S202T02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

Commit message: projektavimas
Parts:
- removed Q1: (no value), crystal:HC18U-V
- added X9: 16MHz, SparkFun:HC49US
Connections:
- removed net 0(RX0): U$2.2
- removed net 1(TX0): U$2.3
- removed net N$3: Q1.2
- net +5V: no longer IC2.16, U$2.16, USB.VBUS, X10.3
- net D8(RX0): now also U$2.2
- net D9(TX0): now also U$2.3
- net N$1: now also X9.1; no longer Q1.1
- net N$2: now also X9.2
- net VCC: now also IC2.16, U$2.16, USB.VBUS, X10.3
Changed lines of the file:
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@@
 </variantdefs>
 <classes>
-<class number="0" name="default" width="0.5" drill="0">
+<class number="0" name="default" width="0.1778" drill="0">
+<clearance class="0" value="0.205"/>
 </class>
 <class number="1" name="power" width="0.6096" drill="0">
@@
 <attribute name="OC_FARNELL" value="1462926" x="96.52" y="2.54" size="1.778" layer="27" rot="R180" display="off"/>
 </element>
-<element name="Q1" library="crystal" package="HC18U-V" value="" x="41.91" y="71.12">
-<attribute name="OC_NEWARK" value="unknown" x="41.91" y="71.12" size="1.778" layer="27" display="off"/>
-<attribute name="MPN" value="" x="41.91" y="71.12" size="1.778" layer="27" display="off"/>
-<attribute name="MF" value="" x="41.91" y="71.12" size="1.778" layer="27" display="off"/>
-<attribute name="OC_FARNELL" value="unknown" x="41.91" y="71.12" size="1.778" layer="27" display="off"/>
-</element>
+<element name="X9" library="SparkFun" package="HC49US" value="16MHz" x="40.64" y="67.31"/>
 </elements>
 <signals>
@@
 <contactref element="R15" pad="2"/>
 <contactref element="C13" pad="1"/>
-<wire x1="-13.97" y1="104.14" x2="46.99" y2="63.5" width="0" layer="19" extent="1-1"/>
+<contactref element="U$2" pad="16"/>
+<contactref element="USB" pad="VBUS"/>
+<contactref element="X10" pad="3"/>
+<contactref element="IC2" pad="16"/>
+<wire x1="120.65" y1="69.85" x2="153.67" y2="83.82" width="0" layer="19" extent="1-1"/>
+<wire x1="110.49" y1="19.05" x2="120.65" y2="69.85" width="0" layer="19" extent="1-1"/>
+<wire x1="46.99" y1="63.5" x2="120.65" y2="69.85" width="0" layer="19" extent="1-1"/>
+<wire x1="10.795" y1="72.65" x2="46.99" y2="63.5" width="0" layer="19" extent="1-1"/>
+<wire x1="7.18" y1="79.07" x2="10.795" y2="72.65" width="0" layer="19" extent="1-1"/>
+<wire x1="-13.97" y1="104.14" x2="7.18" y2="79.07" width="0" layer="19" extent="1-1"/>
 <wire x1="-16.51" y1="120.65" x2="-13.97" y2="104.14" width="0" layer="19" extent="1-1"/>
-<wire x1="153.67" y1="83.82" x2="-16.51" y2="120.65" width="0" layer="19" extent="1-1"/>
-<wire x1="-36.83" y1="120.65" x2="153.67" y2="83.82" width="0" layer="19" extent="1-1"/>
+<wire x1="-36.83" y1="120.65" x2="-16.51" y2="120.65" width="0" layer="19" extent="1-1"/>
 <wire x1="-49.53" y1="109.22" x2="-36.83" y2="120.65" width="0" layer="19" extent="1-1"/>
 <wire x1="-52.07" y1="109.22" x2="-49.53" y2="109.22" width="0" layer="19" extent="1-1"/>
+<wire x1="-63.5" y1="97.79" x2="-52.07" y2="109.22" width="0" layer="19" extent="1-1"/>
+<wire x1="-72.39" y1="97.79" x2="-63.5" y2="97.79" width="0" layer="19" extent="1-1"/>
+<wire x1="-69.85" y1="85.09" x2="-72.39" y2="97.79" width="0" layer="19" extent="1-1"/>
 <wire x1="-67.31" y1="115.57" x2="-52.07" y2="109.22" width="0" layer="19" extent="1-1"/>
-<wire x1="-72.39" y1="97.79" x2="-67.31" y2="115.57" width="0" layer="19" extent="1-1"/>
-<wire x1="-69.85" y1="85.09" x2="-72.39" y2="97.79" width="0" layer="19" extent="1-1"/>
-<wire x1="16.51" y1="35.56" x2="-69.85" y2="85.09" width="0" layer="19" extent="1-1"/>
-<wire x1="120.65" y1="69.85" x2="16.51" y2="35.56" width="0" layer="19" extent="1-1"/>
 <wire x1="-97.79" y1="97.79" x2="-72.39" y2="97.79" width="0" layer="19" extent="1-1"/>
+<wire x1="16.51" y1="35.56" x2="10.795" y2="72.65" width="0" layer="19" extent="1-1"/>
 </signal>
 <signal name="N$1">
 <contactref element="IC4" pad="13"/>
 <contactref element="C11" pad="1"/>
-<contactref element="Q1" pad="1"/>
-<wire x1="39.37" y1="63.5" x2="36.83" y2="77.47" width="0" layer="19" extent="1-1"/>
-<wire x1="39.37" y1="71.12" x2="39.37" y2="63.5" width="0" layer="19" extent="1-1"/>
+<contactref element="X9" pad="1"/>
+<wire x1="39.37" y1="63.5" x2="38.1" y2="67.31" width="0" layer="19" extent="1-1"/>
+<wire x1="36.83" y1="77.47" x2="39.37" y2="63.5" width="0" layer="19" extent="1-1"/>
 </signal>
 <signal name="N$2">
 <contactref element="IC4" pad="12"/>
 <contactref element="C10" pad="1"/>
+<contactref element="X9" pad="2"/>
 <wire x1="41.91" y1="63.5" x2="41.91" y2="76.2" width="0" layer="19" extent="1-1"/>
+<wire x1="43.18" y1="67.31" x2="41.91" y2="63.5" width="0" layer="19" extent="1-1"/>
 </signal>
 <signal name="N$8">
@@
 <contactref element="IC4" pad="7"/>
 </signal>
-<signal name="1(TX0)">
-<contactref element="U$2" pad="3"/>
-</signal>
 <signal name="D11(TX1)">
 <contactref element="IC4" pad="17"/>
-</signal>
-<signal name="0(RX0)">
-<contactref element="U$2" pad="2"/>
 </signal>
 <signal name="D102(RX1)">
@@
 <contactref element="JP5" pad="3"/>
 <contactref element="JP6" pad="2"/>
-<contactref element="U$2" pad="16"/>
-<contactref element="USB" pad="VBUS"/>
-<contactref element="X10" pad="3"/>
-<contactref element="IC2" pad="16"/>
-<wire x1="7.18" y1="79.07" x2="18.8214" y2="26.0604" width="0" layer="19" extent="1-1"/>
-<wire x1="10.795" y1="72.65" x2="7.18" y2="79.07" width="0" layer="19" extent="1-1"/>
-<wire x1="-63.5" y1="97.79" x2="10.795" y2="72.65" width="0" layer="19" extent="1-1"/>
-<wire x1="19.05" y1="35.56" x2="10.795" y2="72.65" width="0" layer="19" extent="1-1"/>
-<wire x1="17.78" y1="39.37" x2="19.05" y2="35.56" width="0" layer="19" extent="1-1"/>
-<wire x1="110.49" y1="19.05" x2="17.78" y2="39.37" width="0" layer="19" extent="1-1"/>
-<wire x1="-85.05" y1="115.57" x2="-63.5" y2="97.79" width="0" layer="19" extent="1-1"/>
+<wire x1="19.05" y1="35.56" x2="17.78" y2="39.37" width="0" layer="19" extent="1-1"/>
+<wire x1="18.8214" y1="26.0604" x2="19.05" y2="35.56" width="0" layer="19" extent="1-1"/>
+<wire x1="-85.05" y1="115.57" x2="17.78" y2="39.37" width="0" layer="19" extent="1-1"/>
 </signal>
 <signal name="N$14">
@@
 <signal name="D9(TX0)">
 <contactref element="IC4" pad="15"/>
+<contactref element="U$2" pad="3"/>
+<wire x1="13.335" y1="67.05" x2="34.29" y2="63.5" width="0" layer="19" extent="1-1"/>
 </signal>
 <signal name="D8(RX0)">
 <contactref element="IC4" pad="14"/>
+<contactref element="U$2" pad="2"/>
+<wire x1="12.065" y1="67.05" x2="36.83" y2="63.5" width="0" layer="19" extent="1-1"/>
 </signal>
 <signal name="D7(SCK)">
@@
 <contactref element="U$1" pad="P$10"/>
 </signal>
-<signal name="N$3">
-<contactref element="Q1" pad="2"/>
-</signal>
 </signals>

Commit message: projektavimas
Parts:
- moved Y1 17.6 mm to (21.6, 78.7), turned to 90 degrees
- moved C11 15.3 mm to (43.2, 63.5), turned to 180 degrees
- moved C10 13.3 mm to (45.7, 63.5)
- moved IC3 12.8 mm to (8.89, 29.2)
- moved C3 7.41 mm to (20.3, 71.1), turned to 90 degrees
- moved U$2 6.35 mm to (15.2, 76.2), turned to 90 degrees
- moved IC4 5.39 mm to (49.5, 52.1)
- moved C17 5.24 mm to (8.89, 71.1), turned to 180 degrees
- moved X9 2.84 mm to (43.2, 68.6)

Commit message: projektavimas
Parts:
- removed D1: BAT85, SteveMarple:DIODE-TH-0.4
- removed R16, R17: 330, resistor-1:0207/10
- added DIODE1: BAT85, SteveMarple:DIODE-TH-0.4
- added R1: 330, resistor-1:0207/10
- added R10: 1k, SteveMarple:RES-AXIAL-0.4
- added R13: 2.2k, adafruit:0207/10
- BAT1: value CR2032 -> (none); device SparkFun:BATTCOM_20MM_PTH -> SparkFun-Electromechanical:BATTCOM_20MM_PTH
- R15: value 2.2k -> 4.7K
- R2: value 1k -> 330; device SteveMarple:RES-AXIAL-0.4 -> resistor-1:0207/10
- R6: value 10k -> 330; device SteveMarple:RES-AXIAL-0.4 -> resistor-1:0207/10
- R7: value 330 -> 10k; device resistor-1:0207/10 -> SteveMarple:RES-AXIAL-0.4
- moved R12 238.7 mm to (121.9, 21.6)
- moved R5 174.9 mm to (72.4, 27.9), turned to 270 degrees
- moved R2 167.6 mm to (49.5, 27.9), turned to 270 degrees
- moved R4 156.9 mm to (64.8, 27.9), turned to 270 degrees
- moved X10 148.7 mm to (82.5, 91.4)
- moved R15 142.2 mm to (82.5, 82.5), turned to 90 degrees
- moved R3 139.5 mm to (57.1, 27.9), turned to 270 degrees
- moved R7 129.1 mm to (2.54, 22.9)
- moved L1 128.1 mm to (33.0, 33.0)
- moved C6 125.2 mm to (24.1, 3.81)
- moved R6 125.0 mm to (80.0, 27.9), turned to 270 degrees
- moved LED2 116.8 mm to (0.00, 26.7)
- moved IC5 111.2 mm to (14.0, 53.3)
- moved Q4 108.0 mm to (14.0, 55.9)
- moved BAT1 107.3 mm to (27.9, 47.0)
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- renumbered D3 to DIODE2
Connections:
- net !RESET: now also DIODE1.A, R7.P$1; no longer D1.A, R6.P$1
- net D0: now also R1.1; no longer R7.1
- net D1: now also R2.1; no longer R4.1
- net D17(SDA): now also R13.1; no longer R15.1
- net D2: now also R15.2
- net D3: now also R4.1; no longer R5.1
- net D4: now also R5.1; no longer R17.1
- net D5: now also R6.1; no longer R16.1
- net N$24: now also R2.2; no longer R4.2
- net N$28: now also R4.2; no longer R5.2
- net N$31: now also R1.2; no longer R7.2
- net N$34: now also R6.2; no longer R16.2
- net N$37: now also R5.2; no longer R17.2
- net N$8: now also R10.P$1; no longer R2.P$1
- net VCC: now also DIODE1.C, R10.P$2, R13.2, R15.1, R7.P$2; no longer D1.C, R15.2, R2.P$2, R6.P$2

Commit message: projektavimas
Parts:
- removed C1, C2, C8: 1u, SparkFun:CAP-PTH-5MM
- removed IC1: MCP1702-3.3, burr-brown:SOT223
- removed IC3: MCP1702-5.0, burr-brown:SOT223
- removed JP5: 3V3/5V, SparkFun:1X03
- removed JP6: VREG PWR, SparkFun:1X02
- moved R15 109.3 mm to (-26.7, 87.6)
- moved X10 104.4 mm to (-21.6, 99.1)
- moved C5 102.3 mm to (-17.8, 72.4)
- moved Q4 92.7 mm to (106.7, 53.3), turned to 270 degrees
- moved U$1 88.7 mm to (85.1, 99.1), turned to 180 degrees
- moved IC5 86.4 mm to (100.3, 55.9), turned to 90 degrees
- moved S1 68.6 mm to (101.6, 81.3), turned to 270 degrees
- moved BAT1 54.7 mm to (-26.7, 49.5)
- moved C13 54.0 mm to (-10.2, 73.7)
- moved S2 47.0 mm to (109.2, 91.4), turned to 90 degrees
- moved R9 46.0 mm to (110.5, 99.1)
- moved C9 43.4 mm to (-6.35, 80.0)
- moved R8 40.9 mm to (97.8, 99.1), turned to 180 degrees
- moved S4 39.5 mm to (101.6, 91.4), turned to 270 degrees
- moved C7 36.1 mm to (-5.08, 86.4)
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Connections:
- removed net +5V: C1.1, IC1.3, JP5.3, JP6.2
- removed net D10: U$1.P$11
- removed net D102(RX1): IC4.16
- removed net D11: U$1.P$10
- removed net D6: IC2.2, R12.1
- removed net D7: IC2.7
- removed net D8: IC2.15
- removed net D9: IC2.10
- removed net N$14: IC3.2, JP6.1
- removed net VIN: C8.1, IC3.3
- new net D10(RX1): IC2.7, IC4.16
- net +3V3: no longer C2.1, IC1.2, JP5.1
- net D11(TX1): now also IC2.2
- net D12: now also IC2.10; no longer U$1.P$9
- net D13: now also IC2.15; no longer U$1.P$12
- net D14: now also R12.1; no longer U$1.P$13
- net D15: now also U$1.P$9; no longer U$1.P$14
- net D18(TCK): now also U$1.P$10
- net D19(TMS): now also U$1.P$11
- net D20(TDO): now also U$1.P$12
- net D21: now also U$1.P$13
- net D22: now also U$1.P$14
- net GND: no longer C1.2, C2.2, C8.2, IC1.1, IC3.1
- net VCC: no longer JP5.2
Other:
- board size 160 x 100 mm -> 120 x 100 mm

Commit message: projektavimas
Parts:
- X10: value (none) -> 22-23-2031; device con-phoenix-254:3POL254 -> con-molex:22-23-2031
- moved X10 136.5 mm to (74.9, 2.54)
- moved C5 128.9 mm to (110.5, 59.7)
- moved R15 126.5 mm to (76.2, 14.0)
- moved BAT1 124.9 mm to (97.8, 39.4)
- moved C7 95.8 mm to (73.7, 31.8)
- moved C9 66.1 mm to (45.7, 39.4)
- moved C13 51.4 mm to (29.2, 40.6)
- moved DIODE1 20.1 mm to (11.4, 22.9)
- moved R10 14.0 mm to (12.7, 12.7)
- moved C6 13.0 mm to (11.4, 6.35), turned to 180 degrees
- moved K1 12.7 mm to (25.4, 15.2)
- moved K3 12.7 mm to (40.6, 15.2)
- moved K4 12.7 mm to (48.3, 15.2)
- moved K6 12.7 mm to (63.5, 15.2)
- moved R3 12.7 mm to (36.8, 26.7)
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Connections:
- net D2: no longer R15.2, X10.2
- net D6(MISO): now also R15.2, X10.2

Commit message: trasavimas
Parts:
- moved USB 122.6 mm to (121.3, 50.2), turned to 90 degrees
- moved U$2 87.7 mm to (102.9, 46.4), turned to 270 degrees
- moved C3 81.4 mm to (91.4, 47.0), turned to 0 degrees
- moved Y1 71.8 mm to (92.7, 40.6), turned to 270 degrees
- moved C17 37.0 mm to (52.1, 39.4), turned to 90 degrees
- moved R11 30.9 mm to (86.4, 86.4), turned to 90 degrees
- moved BAT1 30.5 mm to (97.8, 69.8)
- moved R9 24.0 mm to (90.2, 86.4), turned to 270 degrees
- moved C5 22.5 mm to (88.9, 53.3)
- moved R14 12.7 mm to (19.1, 59.7)
- moved L1 12.5 mm to (19.1, 67.3)
- moved IC5 12.0 mm to (90.2, 62.2)
- moved S1 12.0 mm to (91.4, 74.9)
- moved DIODE2 11.7 mm to (104.1, 20.3)
- moved Q4 10.9 mm to (97.8, 59.7)
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Connections:
- net N$12 renamed D-
- net N$22 renamed D+
Routing:
- net GND: track 0.00 -> 428.1 mm, vias 0 -> 2
- net VCC: track 0.00 -> 312.3 mm, vias 0 -> 3
- net !RESET: track 0.00 -> 197.5 mm, vias 0 -> 4
- net A0: track 0.00 -> 102.3 mm, vias 0 -> 1
- net AVCC: track 0.00 -> 85.0 mm, vias 0 -> 1
- net D16(SCL): track 0.00 -> 79.2 mm, vias 0 -> 2
- net D5: track 0.00 -> 74.1 mm, vias 0 -> 2
- net D17(SDA): track 0.00 -> 73.0 mm, vias 0 -> 2
- net D6(MISO): track 0.00 -> 64.9 mm, vias 0 -> 3
- net D12: track 0.00 -> 58.4 mm, vias 0 -> 2
- net AREF: track 0.00 -> 48.2 mm, vias 0 -> 1
- net D10(RX1): track 0.00 -> 38.2 mm
- net D22: track 0.00 -> 30.5 mm
- net D14: track 0.00 -> 30.1 mm
- net D0: track 0.00 -> 29.2 mm
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Other:
- outline, holes or cut-outs redrawn

Commit message: trasavimas, išmesta ch340
Parts:
- removed C17: 0.1uF, rcl:C025-024X044
- removed C3: 100n, SparkFun:CAP-PTH-SMALL
- removed U$2: CH340G, ch340:SO016
- removed USB: (no value), adafruit:USB-MINIB-THM-MOLEX
- removed Y1: 12mhz, SparkFun-FreqCtrl:RESONATOR-PTH
- added C1: 22p, SparkFun:CAP-PTH-SMALL
- added JP1: (no value), SparkFun-Connectors-1:1X05
- moved C5 2.54 mm to (88.9, 50.8)
- moved IC5 1.27 mm to (90.2, 61.0)
- moved Q4 1.27 mm to (97.8, 58.4)
Connections:
- removed net D+: U$2.5, USB.D+
- removed net D-: U$2.6, USB.D-
- removed net N$11: C17.1, U$2.14
- removed net N$5: U$2.7, Y1.1
- removed net N$7: C3.2, U$2.4
- removed net N$9: U$2.8, Y1.3
- new net DTR: C1.1, JP1.4
- net !RESET: now also C1.2; no longer C17.2
- net D8(RX0): now also JP1.2; no longer U$2.2
- net D9(TX0): now also JP1.3; no longer U$2.3
- net GND: no longer C3.1, U$2.1, USB.GND, USB.ID, Y1.2
- net VCC: no longer U$2.16, USB.VBUS
Routing:
- net D8(RX0): track 0.00 -> 58.0 mm, vias 0 -> 1
- net D9(TX0): track 0.00 -> 54.7 mm, vias 0 -> 1
- net D17(SDA): track 73.0 -> 119.1 mm, vias 2 -> 0
- net DTR: track 0.00 -> 39.9 mm
- net GND: track 428.1 -> 396.7 mm, vias 2 -> 1
- net VCC: track 312.3 -> 335.4 mm
- net !RESET: track 197.5 -> 181.2 mm, vias 4 -> 1
- net N$7: track 6.09 -> 0.00 mm
- net D14: track 30.1 -> 26.4 mm
- net AREF: track 48.2 -> 50.6 mm, vias 1 -> 0
- net D6(MISO): track 64.9 -> 63.5 mm, vias 3 -> 1
- net D12: track 58.4 -> 57.4 mm
- net N$20: track 5.20 -> 4.41 mm
- net D16(SCL): track 79.2 -> 78.6 mm
- net N$27: track 26.8 -> 27.3 mm

Commit message: trasavimas
Parts:
- added AC-DC-5V: HLK-PM01_AC_DC, HLK-PM01:HLK-PM01_AC_DC
- added C2: (no value), rcl-1:C025-024X044
- added J4: HEAD3X2, MyCON2:HEAD3X2
- added JP2: M02PTH2, SparkFun-Connectors-1:1X02_BIG
- added U$4: 2-3.50, con-phoenix-350-1:2-3.50
- moved C6 98.8 mm to (81.3, 83.8), turned to 180 degrees
- moved DIODE1 85.7 mm to (80.0, 74.3), turned to 90 degrees
- moved R7 84.2 mm to (83.8, 74.3), turned to 90 degrees
- moved R14 73.6 mm to (90.8, 43.2), turned to 90 degrees
- moved R13 72.1 mm to (88.3, 43.2), turned to 270 degrees
- moved U$1 66.2 mm to (19.1, 63.5), turned to 0 degrees
- moved R10 34.6 mm to (6.99, 53.3)
- moved LED2 21.8 mm to (3.17, 58.4), turned to 0 degrees
- moved C7 20.4 mm to (55.2, 40.6), turned to 270 degrees
- moved IC5 15.9 mm to (97.8, 47.0)
- moved Q4 15.9 mm to (105.4, 44.5)
- moved JP1 15.2 mm to (116.8, 58.4), turned to 270 degrees
- moved R1 12.3 mm to (28.6, 36.8), turned to 180 degrees
- moved C5 11.7 mm to (99.1, 56.5)
- moved L1 8.26 mm to (15.9, 59.7)
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Connections:
- removed net +3V3: U$1.P$16
- removed net D5: IC4.6, R6.1
- new net 220V: AC-DC-5V.AC1, U$4.1
- new net D5(MOSI): IC4.6, J4.4, R6.1
- new net N$3: AC-DC-5V.AC0, JP2.P$1
- new net N$4: JP2.P$2, U$4.2
- net !RESET: now also J4.5
- net A0: no longer R11.1, R9.2, S2.1, S2.2
- net A2: now also U$1.P$14
- net A3: now also U$1.P$13
- net A4: now also U$1.P$12
- net A5: now also U$1.P$11
- net A6: now also U$1.P$10
- net A7: now also R11.1, R9.2, S2.1, S2.2
- net D18(TCK): no longer U$1.P$10
- net D19(TMS): no longer U$1.P$11
- net D20(TDO): no longer U$1.P$12
- net D21: no longer U$1.P$13
- net D22: no longer U$1.P$14
- net D6(MISO): now also J4.1
- net D7(SCK): now also J4.3
- net GND: now also AC-DC-5V.-V, C2.2, J4.6
- net VCC: now also AC-DC-5V.+V, C2.1, J4.2, U$1.P$16
Routing:
- net A0: track 102.3 -> 0.00 mm, vias 1 -> 0
- net D17(SDA): track 119.1 -> 24.0 mm
- net A7: track 0.00 -> 93.9 mm
- net !RESET: track 181.2 -> 98.1 mm
- net D5: track 74.1 -> 0.00 mm, vias 2 -> 0
- net VCC: track 335.4 -> 265.3 mm, vias 3 -> 0
- net D16(SCL): track 78.6 -> 24.2 mm, vias 2 -> 0
- net D5(MOSI): track 0.00 -> 52.2 mm
- net D15: track 21.4 -> 72.6 mm, vias 1 -> 0
- net D6(MISO): track 63.5 -> 112.9 mm
- net A6: track 0.00 -> 38.7 mm
- net A5: track 0.00 -> 35.1 mm
- net A4: track 0.00 -> 31.5 mm
- net D22: track 30.5 -> 0.00 mm
- net D21: track 28.5 -> 0.00 mm
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Other:
- outline, holes or cut-outs redrawn
