File: KKK_valdiklis.brd (EAGLE design)
At the start: 120 x 100 mm, 61 parts, among them IC2 L293D, IC4 ATMEGA1284, IC5 DS1307, J4 HEAD3X2, K1 S202T02, K2 S202T02, K3 S202T02, K4 S202T02, K5 S202T02, K6 S202T02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

Commit message: trasavimas
Parts:
- moved R1 2.54 mm to (28.6, 34.3)
- moved C10 1.65 mm to (61.2, 40.6)
Connections:
- net D8(RX0): now also JP1.3; no longer JP1.2
- net D9(TX0): now also JP1.2; no longer JP1.3
- net GND: now also JP1.1
- net VCC: now also IC2.1, IC2.9
Routing:
- net VCC: track 265.3 -> 289.4 mm
- net D9(TX0): track 57.8 -> 76.9 mm, vias 4 -> 2
- net D8(RX0): track 73.9 -> 61.3 mm
- net GND: track 413.9 -> 424.8 mm
- net D0: track 7.94 -> 10.5 mm
- net N$31: track 13.0 -> 10.5 mm
- net D1: track 15.5 -> 16.9 mm
- net N$2: track 8.92 -> 7.81 mm

Commit message: trasavimas
Parts:
- added X11: +12V, con-molex:22-23-2021
- moved X7 3.81 mm to (85.7, 2.67)
- moved X10 3.68 mm to (75.7, 2.67)
- moved C9 3.01 mm to (48.8, 39.2)
- moved C5 2.67 mm to (99.1, 53.8)
- moved R15 2.29 mm to (75.2, 8.38)
- moved R12 1.40 mm to (104.9, 20.6)
Connections:
- removed net +12V: IC2.8
- new net N$5: IC2.8, X11.2
- net D10(RX1): now also IC2.10; no longer IC2.7
- net D12: now also IC2.7; no longer IC2.10
- net GND: now also X11.1
Routing:
- net D6(MISO): track 112.9 -> 80.9 mm, vias 1 -> 0
- net VCC: track 289.4 -> 264.9 mm
- net GND: track 424.8 -> 449.3 mm
- net D10(RX1): track 48.9 -> 67.1 mm
- net D12: track 51.7 -> 39.1 mm
- net N$5: track 0.00 -> 8.15 mm
- net D9(TX0): track 76.9 -> 73.0 mm, vias 2 -> 1
- net D4: track 16.7 -> 19.4 mm
- net D5(MOSI): track 52.2 -> 54.7 mm
- net AVCC: track 85.1 -> 83.4 mm, vias 2 -> 1
- net AREF: track 49.2 -> 50.3 mm
- net MV1.2: track 14.0 -> 15.1 mm
- net MV1.1: track 21.7 -> 21.8 mm, vias 0 -> 1

Commit message: trasavimas
Parts:
- renumbered Q2 to T2
Connections:
- removed net N$5: IC2.8, X11.2
- new net +12V: IC2.8, X11.2, X77.4
- net N$15: no longer X77.4
Routing:
- net +12V: track 0.00 -> 24.1 mm
- net N$5: track 8.15 -> 0.00 mm, vias 0 -> 1
- net GND: track 449.3 -> 452.3 mm
- net N$15: track 15.7 -> 13.2 mm
Changed lines of the file:
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@@
 <element name="R9" library="resistor" package="0207/10" value="1k" x="92.075" y="89.535" rot="R90"/>
 <element name="R11" library="resistor" package="0207/10" value="2k" x="88.265" y="89.535" rot="R270"/>
-<element name="Q2" library="rocketfarm" package="TO220AV" value="TIP120V" x="108.585" y="14.097"/>
+<element name="T2" library="rocketfarm" package="TO220AV" value="TIP120V" x="108.585" y="14.097"/>
 <element name="X77" library="con-molex" package="22-23-2041" value="PUMP1" x="108.585" y="2.667" rot="R180">
 <attribute name="OC_NEWARK" value="38C0355" x="23.495" y="64.897" size="1.778" layer="27" rot="R180" display="off"/>
@@
 <contactref element="S4" pad="3"/>
 <contactref element="S4" pad="4"/>
-<contactref element="Q2" pad="E"/>
+<contactref element="T2" pad="E"/>
 <contactref element="DIODE2" pad="A"/>
 <contactref element="IC5" pad="4"/>
@@
 <wire x1="89.535" y1="20.447" x2="88.519" y2="20.447" width="0.5" layer="16"/>
 <wire x1="68.7705" y1="31.6865" x2="68.58" y2="31.8135" width="0.5" layer="16"/>
+<wire x1="53.6575" y1="36.703" x2="48.768" y2="36.703" width="0.5" layer="16"/>
+<wire x1="54.991" y1="38.0365" x2="53.6575" y2="36.703" width="0.5" layer="16"/>
+<wire x1="54.991" y1="38.0365" x2="55.245" y2="38.1" width="0.5" layer="16"/>
+<wire x1="73.152" y1="3.175" x2="73.152" y2="2.667" width="0.5" layer="1"/>
+<wire x1="74.803" y1="4.826" x2="73.152" y2="3.175" width="0.5" layer="1"/>
+<wire x1="91.694" y1="4.826" x2="74.803" y2="4.826" width="0.5" layer="1"/>
+<wire x1="93.345" y1="3.175" x2="91.694" y2="4.826" width="0.5" layer="1"/>
+<wire x1="93.345" y1="2.667" x2="93.345" y2="3.175" width="0.5" layer="1"/>
 <wire x1="93.345" y1="14.478" x2="93.345" y2="2.667" width="0.5" layer="16"/>
 <wire x1="96.774" y1="17.907" x2="93.345" y2="14.478" width="0.5" layer="16"/>
 <wire x1="97.155" y1="17.907" x2="96.774" y2="17.907" width="0.5" layer="16"/>
-<wire x1="73.152" y1="2.159" x2="73.152" y2="2.667" width="0.5" layer="16"/>
-<wire x1="74.803" y1="0.508" x2="73.152" y2="2.159" width="0.5" layer="16"/>
-<wire x1="91.694" y1="0.508" x2="74.803" y2="0.508" width="0.5" layer="16"/>
-<wire x1="93.218" y1="2.032" x2="91.694" y2="0.508" width="0.5" layer="16"/>
-<wire x1="93.218" y1="2.4765" x2="93.218" y2="2.032" width="0.5" layer="16"/>
-<wire x1="93.218" y1="2.4765" x2="93.345" y2="2.667" width="0.5" layer="16"/>
-<wire x1="53.6575" y1="36.703" x2="48.768" y2="36.703" width="0.5" layer="16"/>
-<wire x1="54.991" y1="38.0365" x2="53.6575" y2="36.703" width="0.5" layer="16"/>
-<wire x1="54.991" y1="38.0365" x2="55.245" y2="38.1" width="0.5" layer="16"/>
+<wire x1="70.231" y1="2.667" x2="73.152" y2="2.667" width="0.4064" layer="16"/>
 </signal>
 <signal name="VCC" class="1">
@@
 <signal name="N$13">
 <contactref element="R12" pad="2"/>
-<contactref element="Q2" pad="B"/>
+<contactref element="T2" pad="B"/>
 <wire x1="104.902" y1="12.7" x2="104.902" y2="15.494" width="0.4" layer="16"/>
 <wire x1="106.045" y1="11.557" x2="104.902" y2="12.7" width="0.4" layer="16"/>
 </signal>
 <signal name="N$15">
-<contactref element="Q2" pad="C"/>
+<contactref element="T2" pad="C"/>
 <contactref element="DIODE2" pad="C"/>
 <contactref element="X77" pad="3"/>
-<contactref element="X77" pad="4"/>
-<wire x1="107.315" y1="2.667" x2="104.775" y2="2.667" width="0.4" layer="16"/>
 <wire x1="108.585" y1="15.367" x2="108.585" y2="11.557" width="0.4" layer="16"/>
 <wire x1="107.3785" y1="8.382" x2="107.3785" y2="2.8575" width="0.4" layer="16"/>
@@
 <wire x1="14.097" y1="7.1755" x2="14.135" y2="7.182" width="0.5" layer="16"/>
 </signal>
-<signal name="N$5">
+<signal name="+12V">
+<contactref element="X77" pad="4"/>
 <contactref element="IC2" pad="8"/>
 <contactref element="X11" pad="2"/>
 <wire x1="89.535" y1="3.937" x2="89.535" y2="10.287" width="0.4" layer="16"/>
 <wire x1="90.805" y1="2.667" x2="89.535" y2="3.937" width="0.4" layer="16"/>
+<wire x1="102.6795" y1="2.667" x2="104.775" y2="2.667" width="0.4" layer="16"/>
+<wire x1="100.5205" y1="0.508" x2="102.6795" y2="2.667" width="0.4" layer="16"/>
+<wire x1="92.5195" y1="0.508" x2="100.5205" y2="0.508" width="0.4" layer="16"/>
+<wire x1="90.8685" y1="2.159" x2="92.5195" y2="0.508" width="0.4" layer="16"/>
+<wire x1="90.8685" y1="2.4765" x2="90.8685" y2="2.159" width="0.4" layer="16"/>
+<wire x1="90.8685" y1="2.4765" x2="90.805" y2="2.667" width="0.4" layer="16"/>
+</signal>
+<signal name="N$5">
+<via x="70.104" y="2.667" extent="1-16" drill="0.508"/>
 </signal>
 </signals>
