File: KKK_valdiklis.sch (EAGLE design)
At the start: 72 parts, among them IC1 MCP1702-3.3, IC3 MCP1702-5.0, IC4 ATMEGA1284, IC5 DS1307, K1 S202T02, K2 S202T02, K3 S202T02, K4 S202T02, K5 S202T02, K7 S202T02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

Commit message: eiga...
Parts:
- removed X13, X14, X15, X5, X6, X7, X8, X9: (no value), con-phoenix-254:MPT3
Connections:
- net 11(MOSI) renamed D5(MOSI)
- net 12(MISO) renamed D6(MISO)
- net 14 renamed D23
- net 15 renamed D22
- net 16(TDI) renamed D21
- net 17(TDO) renamed D20(TDO)
- net 18(TMS) renamed D19(TMS)
- net 19(TCK) renamed D18(TCK)
- net 2(RX1) renamed D102(RX1)
- net 22 renamed D12
- net 23 renamed D15
- net 3(TX1) renamed D11(TX1)
- net 4 renamed D0
- net 8 renamed D14
- net 9 renamed D13
- removed net 10: IC4.PCINT12/OC0B/SS_PB4
- removed net 5: IC4.PCINT9/CLKO/T1_PB1
- removed net 6: IC4.PCINT10/INT2/AIN0_PB2
- removed net 7: IC4.PCINT11/OC0A/AIN1_PB3
- new net D16(SCL): IC4.PCINT16/SCL_PC0
- new net D17(SDA): IC4.PCINT17/SDA_PC1
- new net D7(SCK): IC4.PCINT15/SCK_PB7
- new net D8(RX0): IC4.PCINT24/RXD0_PD0
- new net D9(TX0): IC4.PCINT25/TXD0_PD1
- net +5V: no longer X13-3.1, X14-3.1, X15-3.1, X5-3.1, X6-3.1, X7-3.1, X8-3.1, X9-3.1
- net 0(RX0): no longer IC4.PCINT24/RXD0_PD0
- net 1(TX0): no longer IC4.PCINT25/TXD0_PD1
- net 13(SCK): no longer IC4.PCINT15/SCK_PB7
- net 20(SDA): no longer IC4.PCINT17/SDA_PC1
- net 21(SCL): no longer IC4.PCINT16/SCL_PC0
- net A0: now also IC4.PCINT0/ADC0_PA0; no longer IC4.PCINT7/ADC7_PA7
- net A1: now also IC4.PCINT1/ADC1_PA1; no longer IC4.PCINT6/ADC6_PA6, X14-2.1, X6-2.1, X9-2.1
- net A2: now also IC4.PCINT2/ADC2_PA2; no longer IC4.PCINT5/ADC5_PA5
- net A3: now also IC4.PCINT3/ADC3_PA3; no longer IC4.PCINT4/ADC4_PA4
- net A4: now also IC4.PCINT4/ADC4_PA4; no longer IC4.PCINT3/ADC3_PA3
- net A5: now also IC4.PCINT5/ADC5_PA5; no longer IC4.PCINT2/ADC2_PA2
- net A6: now also IC4.PCINT6/ADC6_PA6; no longer IC4.PCINT1/ADC1_PA1
- net A7: now also IC4.PCINT7/ADC7_PA7; no longer IC4.PCINT0/ADC0_PA0
- net D1: now also IC4.PCINT9/CLKO/T1_PB1; no longer X13-2.1, X5-2.1, X8-2.1
- net D2: now also IC4.PCINT10/INT2/AIN0_PB2; no longer X15-2.1, X7-2.1
- net D3: now also IC4.PCINT11/OC0A/AIN1_PB3
- net D4: now also IC4.PCINT12/OC0B/SS_PB4
- net GND: no longer X13-1.1, X14-1.1, X15-1.1, X5-1.1, X6-1.1, X7-1.1, X8-1.1, X9-1.1

Commit message: projektavimas
Parts:
- added IC2: L293D, st-microelectronics:L293D
Connections:
- removed net D6: R4.1
- removed net D7: R7.1
- removed net D8: R16.1
- removed net D9: R17.1
- net D0: now also R5.1
- net D1: now also R17.1
- net D2: now also R16.1
- net D3: now also R7.1
- net D4: now also R4.1; no longer R3.1
- net D5: now also R3.1; no longer R5.1
Changed lines of the file:
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@@
 <part name="R17" library="resistor-1" deviceset="R-US_" device="0207/10" value="330"/>
 <part name="GND13" library="SparkFun-Aesthetics" deviceset="GND" device=""/>
+<part name="IC2" library="st-microelectronics" deviceset="L293D" device=""/>
 </parts>
 <sheets>
@@
 </instance>
 <instance part="GND13" gate="1" x="-2.54" y="127"/>
+<instance part="IC2" gate="G$1" x="-58.42" y="137.16"/>
 </instances>
 <busses>
@@
 <pinref part="IC4" gate="G$1" pin="PCINT8/XCK0/T0_PB0"/>
 </segment>
+<segment>
+<pinref part="R5" gate="G$1" pin="1"/>
+<wire x1="-10.16" y1="152.4" x2="-20.32" y2="152.4" width="0.1524" layer="91"/>
+<label x="-20.32" y="154.94" size="1.778" layer="95"/>
+</segment>
 </net>
 <net name="D1" class="0">
@@
 <label x="-17.78" y="30.48" size="1.778" layer="95" rot="MR0"/>
 <pinref part="IC4" gate="G$1" pin="PCINT9/CLKO/T1_PB1"/>
+</segment>
+<segment>
+<pinref part="R17" gate="G$1" pin="1"/>
+<wire x1="-10.16" y1="134.62" x2="-20.32" y2="134.62" width="0.1524" layer="91"/>
+<label x="-20.32" y="137.16" size="1.778" layer="95"/>
 </segment>
 </net>
@@
 <pinref part="IC4" gate="G$1" pin="PCINT11/OC0A/AIN1_PB3"/>
 </segment>
+<segment>
+<pinref part="R7" gate="G$1" pin="1"/>
+<wire x1="45.72" y1="152.4" x2="35.56" y2="152.4" width="0.1524" layer="91"/>
+<label x="35.56" y="154.94" size="1.778" layer="95"/>
+</segment>
 </net>
 <net name="N$13" class="0">
@@
 <pinref part="IC4" gate="G$1" pin="PCINT10/INT2/AIN0_PB2"/>
 </segment>
+<segment>
+<pinref part="R16" gate="G$1" pin="1"/>
+<wire x1="-10.16" y1="116.84" x2="-20.32" y2="116.84" width="0.1524" layer="91"/>
+<label x="-20.32" y="119.38" size="1.778" layer="95"/>
+</segment>
 </net>
 <net name="N$5" class="0">
@@
 </segment>
 </net>
-<net name="D5" class="0">
-<segment>
-<pinref part="R5" gate="G$1" pin="1"/>
-<wire x1="-10.16" y1="152.4" x2="-20.32" y2="152.4" width="0.1524" layer="91"/>
-</segment>
-</net>
 <net name="N$28" class="0">
 <segment>
@@
 <net name="D4" class="0">
 <segment>
-<pinref part="R3" gate="G$1" pin="1"/>
-<wire x1="45.72" y1="114.3" x2="35.56" y2="114.3" width="0.1524" layer="91"/>
-</segment>
-<segment>
 <wire x1="-7.62" y1="22.86" x2="-15.24" y2="22.86" width="0.1524" layer="91"/>
 <label x="-17.78" y="22.86" size="1.778" layer="95" rot="MR0"/>
 <pinref part="IC4" gate="G$1" pin="PCINT12/OC0B/SS_PB4"/>
 </segment>
+<segment>
+<pinref part="R4" gate="G$1" pin="1"/>
+<wire x1="45.72" y1="134.62" x2="35.56" y2="134.62" width="0.1524" layer="91"/>
+<label x="35.56" y="137.16" size="1.778" layer="95"/>
+</segment>
 </net>
 <net name="N$16" class="0">
@@
 </segment>
 </net>
-<net name="D6" class="0">
-<segment>
-<pinref part="R4" gate="G$1" pin="1"/>
-<wire x1="45.72" y1="134.62" x2="35.56" y2="134.62" width="0.1524" layer="91"/>
-</segment>
-</net>
 <net name="N$24" class="0">
 <segment>
@@
 </segment>
 </net>
-<net name="D7" class="0">
-<segment>
-<pinref part="R7" gate="G$1" pin="1"/>
-<wire x1="45.72" y1="152.4" x2="35.56" y2="152.4" width="0.1524" layer="91"/>
-</segment>
-</net>
 <net name="N$31" class="0">
 <segment>
@@
 </segment>
 </net>
-<net name="D8" class="0">
-<segment>
-<pinref part="R16" gate="G$1" pin="1"/>
-<wire x1="-10.16" y1="116.84" x2="-20.32" y2="116.84" width="0.1524" layer="91"/>
-</segment>
-</net>
 <net name="N$34" class="0">
 <segment>
@@
 </segment>
 </net>
-<net name="D9" class="0">
-<segment>
-<pinref part="R17" gate="G$1" pin="1"/>
-<wire x1="-10.16" y1="134.62" x2="-20.32" y2="134.62" width="0.1524" layer="91"/>
-</segment>
-</net>
 <net name="N$37" class="0">
 <segment>
@@
 </segment>
 </net>
+<net name="D5" class="0">
+<segment>
+<pinref part="R3" gate="G$1" pin="1"/>
+<wire x1="45.72" y1="114.3" x2="35.56" y2="114.3" width="0.1524" layer="91"/>
+<label x="35.56" y="116.84" size="1.778" layer="95"/>
+</segment>
+</net>

Commit message: projektavimas
Parts:
- removed K7: S202T02, relay-1:S202T02
- removed LED1: D13, SparkFun:LED3MM
- removed Q1: 2N7000, SteveMarple:2N7000
- removed R1: 1k, SteveMarple:RESISTOR
- removed R10: 1M, SteveMarple:RESISTOR
- added K6: S202T02, relay-1:S202T02
- added X2: Storage tank pump, con-molex:22-23-2021
- added X3: Radiator pump, con-molex:22-23-2021
- added X5: 4 way valve 2, con-molex:22-23-2021
- added X6: Floor heating, con-molex:22-23-2021
- added X77: PUMP1, con-molex:22-23-2041
- added X88: PUMP2, con-molex:22-23-2041
- X1: value PUMP -> Boiler pump; device con-molex:22-23-2041 -> con-molex:22-23-2021
- X4: value PUMP -> 4 way valve 1; device con-molex:22-23-2041 -> con-molex:22-23-2021
Connections:
- removed net 13(SCK): Q1.G, R10.2
- removed net 20(SDA): IC5.SDA, R15.1
- removed net 21(SCL): IC5.SCL, R14.2
- removed net D5(MOSI): IC4.PCINT13/MOSI_PB5
- removed net N$3: LED1.A, R1.1
- removed net N$4: LED1.C, Q1.D
- new net +12V: IC2.VCC2
- new net D6: IC2.1A, R12.1
- new net D7: IC2.2A, R13.1
- new net D8: IC2.4A
- new net D9: IC2.3A
- new net MV1.1: IC2.1Y
- new net MV1.2: IC2.2Y
- new net MV2.1: IC2.4Y
- new net MV2.2: IC2.3Y
- net +5V: now also IC2.VCC1
- net D0: now also R7.1; no longer R5.1
- net D1: now also R4.1; no longer R17.1
- net D16(SCL): now also IC5.SCL, R14.2
- net D17(SDA): now also IC5.SDA, R15.1
- net D2: now also R3.1; no longer R16.1
- net D3: now also R5.1; no longer R12.1, R13.1, R7.1
- net D4: now also R17.1; no longer R4.1
- net D5: now also IC4.PCINT13/MOSI_PB5, R16.1; no longer R3.1
- net GND: now also IC2.GND1, IC2.GND2, IC2.GND3, IC2.GND4, K6.K, X77-3.S, X77-4.S; no longer K7.K, Q1.S, R10.1, X4-3.S, X4-4.S
- net GND1: now also X88-3.S, X88-4.S; no longer X1-3.S, X1-4.S
- net N$15: now also X77-1.S, X77-2.S; no longer X4-1.S, X4-2.S
- net N$16: now also K3.A; no longer K1.A
- net N$18: now also K3.DS1, X3-1.S; no longer K1.DS1
- net N$19: now also X88-1.S, X88-2.S; no longer X1-1.S, X1-2.S
- net N$23: now also K3.DS2, X3-2.S; no longer K1.DS2
- net N$25: now also X2-1.S
- net N$26: now also X2-2.S
- net N$28: now also K4.A; no longer K7.A
- net N$29: now also K4.DS1, X4-1.S; no longer K7.DS1
- net N$30: now also K4.DS2, X4-2.S; no longer K7.DS2
- net N$31: now also K1.A; no longer K3.A
- net N$32: now also K1.DS1, X1-1.S; no longer K3.DS1
- net N$33: now also K1.DS2, X1-2.S; no longer K3.DS2
- net N$34: now also K6.A; no longer K4.A
- net N$35: now also K6.DS1, X6-1.S; no longer K4.DS1
- net N$36: now also K6.DS2, X6-2.S; no longer K4.DS2
- net N$38: now also X5-1.S
- net N$39: now also X5-2.S
- net VCC: no longer R1.2
Other:
- note added: "12V 2A switches"
- note added: "12V motorized valves switch"
- note added: "230V 2A switches"
- note added: "Connector for DS18B20 sensors"
- note removed: "D13 LED"
- note removed: "Onboard peripherals"
- note removed: "Temperaturos jutikliu pajungimo kontaktai"
- moved on the sheet: D3, D4, K1, K2, K3, K4, K5, Q2, Q3, R12, R13, R16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

Commit message: projektavimas
Parts:
- added X7: motorized valve 1, con-molex:22-23-2021
- added X8: motorized valve 2, con-molex:22-23-2021
Connections:
- net MV1.1: now also X7-1.S
- net MV1.2: now also X7-2.S
- net MV2.1: now also X8-1.S
- net MV2.2: now also X8-2.S
Other:
- moved on the sheet: C8, D1, D3, D4, IC3, JP5, JP6, Q2, Q3, R12, R13, R6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

Commit message: projektavimas
Parts:
- removed D4: 1N4004, diode:1N4004
- removed Q3: TIP120V, rocketfarm:TIP120V
- removed R13: 2k, resistor:R-EU_0207/10
- removed X88: PUMP2, con-molex:22-23-2041
- C17: device rcl:C-USC0805K -> rcl:C-EU025-024X044
Connections:
- removed net GND1: D4.A, Q3.E, X88-3.S, X88-4.S
- removed net N$17: Q3.B, R13.2
- removed net N$19: D4.C, Q3.C, X88-1.S, X88-2.S
- new net D10: U$1.SDA
- new net D11: U$1.SCK
- net +3V3: now also U$1.3.3V
- net D12: now also U$1.LED
- net D13: now also U$1.A0
- net D14: now also U$1.RST
- net D15: now also U$1.CS
- net D7: no longer R13.1
- net GND: now also U$1.GND, X77-1.S, X77-2.S; no longer X77-3.S, X77-4.S
- net N$15: now also X77-3.S, X77-4.S; no longer X77-1.S, X77-2.S
Other:
- moved on the sheet: U$1, X77-1, X77-2, X77-3, X77-4
Changed lines of the file:
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@@
 <?xml version="1.0" encoding="utf-8"?>
 <!DOCTYPE eagle SYSTEM "eagle.dtd">
-<eagle version="6.4">
+<eagle version="6.5.0">
 <drawing>
 <settings>
@@
 <part name="R12" library="resistor" deviceset="R-EU_" device="0207/10" value="2k"/>
 <part name="D3" library="diode" deviceset="1N4004" device=""/>
-<part name="Q3" library="rocketfarm" deviceset="TIP120" device="V"/>
-<part name="X88" library="con-molex" deviceset="22-23-2041" device="" value="PUMP2"/>
-<part name="R13" library="resistor" deviceset="R-EU_" device="0207/10" value="2k"/>
-<part name="D4" library="diode" deviceset="1N4004" device=""/>
 <part name="Q4" library="crystal" deviceset="CRYTAL" device="TC38H" value="32.768"/>
 <part name="IC5" library="adafruit" deviceset="DS1307" device=""/>
@@
 <part name="GND5" library="SparkFun" deviceset="GND" device=""/>
 <part name="U$2" library="ch340" deviceset="CH340G" device=""/>
-<part name="C17" library="rcl" deviceset="C-US" device="C0805K" value="0.1uF"/>
+<part name="C17" library="rcl" deviceset="C-EU" device="025-024X044" value="0.1uF"/>
 <part name="+3V9" library="supply1" deviceset="+5V" device=""/>
 <part name="Y1" library="SparkFun-FreqCtrl" deviceset="RESONATOR" device="PTH" value="12mhz"/>
@@
 <part name="X7" library="con-molex" deviceset="22-23-2021" device="" value="motorized valve 1"/>
 <part name="X8" library="con-molex" deviceset="22-23-2021" device="" value="motorized valve 2"/>
+<part name="+3V2" library="supply1" deviceset="+3V3" device=""/>
+<part name="GND3" library="supply1" deviceset="GND" device=""/>
 </parts>
 <sheets>
@@
 <instance part="R11" gate="G$1" x="175.26" y="22.86" rot="R90"/>
 <instance part="Q2" gate="1" x="-76.2" y="76.2"/>
-<instance part="X77" gate="-1" x="-40.64" y="76.2"/>
-<instance part="X77" gate="-2" x="-40.64" y="73.66"/>
-<instance part="X77" gate="-3" x="-40.64" y="71.12"/>
-<instance part="X77" gate="-4" x="-40.64" y="68.58"/>
+<instance part="X77" gate="-1" x="-46.99" y="71.12"/>
+<instance part="X77" gate="-2" x="-46.99" y="68.58"/>
+<instance part="X77" gate="-3" x="-46.99" y="81.28"/>
+<instance part="X77" gate="-4" x="-46.99" y="78.74"/>
 <instance part="R12" gate="G$1" x="-83.82" y="76.2" smashed="yes">
 <attribute name="NAME" x="-87.63" y="77.6986" size="1.778" layer="95"/>
@@
 </instance>
 <instance part="D3" gate="1" x="-58.42" y="73.66" rot="R90"/>
-<instance part="Q3" gate="1" x="-76.2" y="60.96"/>
-<instance part="X88" gate="-1" x="-40.64" y="60.96"/>
-<instance part="X88" gate="-2" x="-40.64" y="58.42"/>
-<instance part="X88" gate="-3" x="-40.64" y="55.88"/>
-<instance part="X88" gate="-4" x="-40.64" y="53.34"/>
-<instance part="R13" gate="G$1" x="-83.82" y="60.96" smashed="yes">
-<attribute name="NAME" x="-87.63" y="62.4586" size="1.778" layer="95"/>
-<attribute name="VALUE" x="-82.55" y="62.738" size="1.778" layer="96"/>
-</instance>
-<instance part="D4" gate="1" x="-58.42" y="58.42" rot="R90"/>
 <instance part="Q4" gate="G$1" x="142.24" y="91.44" rot="R180"/>
 <instance part="IC5" gate="G$1" x="144.78" y="68.58"/>
@@
 <attribute name="VALUE" x="-30.48" y="-52.07" size="1.778" layer="96" rot="R180"/>
 </instance>
-<instance part="U$1" gate="G$1" x="-144.78" y="29.21" rot="R270"/>
+<instance part="U$1" gate="G$1" x="-134.62" y="29.21" rot="R270"/>
 <instance part="K4" gate="G$1" x="7.62" y="111.76"/>
 <instance part="R5" gate="G$1" x="-10.16" y="114.3" smashed="yes">
@@
 </instance>
 <instance part="X8" gate="-2" x="-44.45" y="102.87"/>
+<instance part="+3V2" gate="G$1" x="-154.94" y="21.59" rot="R90"/>
+<instance part="GND3" gate="1" x="-160.02" y="21.59"/>
 </instances>
 <busses>
@@
 <pinref part="D3" gate="1" pin="A"/>
 <wire x1="-58.42" y1="71.12" x2="-58.42" y2="68.58" width="0.1524" layer="91"/>
-<wire x1="-58.42" y1="68.58" x2="-50.8" y2="68.58" width="0.1524" layer="91"/>
-<wire x1="-50.8" y1="68.58" x2="-50.8" y2="71.12" width="0.1524" layer="91"/>
-<pinref part="X77" gate="-3" pin="S"/>
-<wire x1="-50.8" y1="71.12" x2="-43.18" y2="71.12" width="0.1524" layer="91"/>
-<pinref part="X77" gate="-4" pin="S"/>
-<wire x1="-43.18" y1="71.12" x2="-43.18" y2="68.58" width="0.1524" layer="91"/>
+<wire x1="-58.42" y1="68.58" x2="-49.53" y2="68.58" width="0.1524" layer="91"/>
+<pinref part="X77" gate="-2" pin="S"/>
+<pinref part="X77" gate="-1" pin="S"/>
+<wire x1="-49.53" y1="68.58" x2="-49.53" y2="71.12" width="0.1524" layer="91"/>
 </segment>
 <segment>
@@
 <wire x1="-40.64" y1="137.16" x2="-43.18" y2="137.16" width="0.1524" layer="91"/>
 </segment>
+<segment>
+<pinref part="U$1" gate="G$1" pin="GND"/>
+<pinref part="GND3" gate="1" pin="GND"/>
+<wire x1="-147.32" y1="24.13" x2="-160.02" y2="24.13" width="0.1524" layer="91"/>
+</segment>
 </net>
 <net name="VCC" class="1">
@@
 <pinref part="IC4" gate="G$1" pin="PCINT28/OC1B_PD4"/>
 </segment>
+<segment>
+<pinref part="U$1" gate="G$1" pin="LED"/>
+<wire x1="-147.32" y1="39.37" x2="-152.4" y2="39.37" width="0.1524" layer="91"/>
+<label x="-154.94" y="39.37" size="1.778" layer="95"/>
+</segment>
 </net>
 <net name="D13" class="0">
@@
 <pinref part="IC4" gate="G$1" pin="PCINT29/OC1A_PD5"/>
 </segment>
+<segment>
+<pinref part="U$1" gate="G$1" pin="A0"/>
+<wire x1="-147.32" y1="31.75" x2="-152.4" y2="31.75" width="0.1524" layer="91"/>
+<label x="-154.94" y="31.75" size="1.778" layer="95"/>
+</segment>
 </net>
 <net name="D14" class="0">
@@
 <pinref part="IC4" gate="G$1" pin="PCINT30/OC2B/ICP_PD6"/>
 </segment>
+<segment>
+<pinref part="U$1" gate="G$1" pin="RST"/>
+<wire x1="-147.32" y1="29.21" x2="-152.4" y2="29.21" width="0.1524" layer="91"/>
+<label x="-154.94" y="29.21" size="1.778" layer="95"/>
+</segment>
 </net>
 <net name="D0" class="0">
@@
 <label x="58.42" y="-15.24" size="1.778" layer="95"/>
 <pinref part="IC4" gate="G$1" pin="PCINT31/OC2A_PD7"/>
+</segment>
+<segment>
+<pinref part="U$1" gate="G$1" pin="CS"/>
+<wire x1="-147.32" y1="26.67" x2="-152.4" y2="26.67" width="0.1524" layer="91"/>
+<label x="-154.94" y="26.67" size="1.778" layer="95"/>
 </segment>
 </net>
@@
 <pinref part="+3V1" gate="G$1" pin="+3V3"/>
 <pinref part="JP5" gate="G$1" pin="1"/>
+</segment>
+<segment>
+<pinref part="U$1" gate="G$1" pin="3.3V"/>
+<wire x1="-147.32" y1="21.59" x2="-152.4" y2="21.59" width="0.1524" layer="91"/>
+<pinref part="+3V2" gate="G$1" pin="+3V3"/>
 </segment>
 </net>
@@
 <pinref part="Q2" gate="1" pin="C"/>
 <wire x1="-73.66" y1="81.28" x2="-58.42" y2="81.28" width="0.1524" layer="91"/>
-<wire x1="-58.42" y1="81.28" x2="-50.8" y2="81.28" width="0.1524" layer="91"/>
-<wire x1="-50.8" y1="81.28" x2="-50.8" y2="73.66" width="0.1524" layer="91"/>
+<wire x1="-58.42" y1="81.28" x2="-49.53" y2="81.28" width="0.1524" layer="91"/>
 <pinref part="D3" gate="1" pin="C"/>
 <wire x1="-58.42" y1="76.2" x2="-58.42" y2="81.28" width="0.1524" layer="91"/>
-<pinref part="X77" gate="-2" pin="S"/>
-<wire x1="-50.8" y1="73.66" x2="-43.18" y2="73.66" width="0.1524" layer="91"/>
-<pinref part="X77" gate="-1" pin="S"/>
-<wire x1="-43.18" y1="76.2" x2="-43.18" y2="73.66" width="0.1524" layer="91"/>
-</segment>
-</net>
-<net name="GND1" class="1">
-<segment>
-<pinref part="Q3" gate="1" pin="E"/>
-<wire x1="-73.66" y1="55.88" x2="-73.66" y2="53.34" width="0.1524" layer="91"/>
-<wire x1="-73.66" y1="53.34" x2="-58.42" y2="53.34" width="0.1524" layer="91"/>
-<pinref part="D4" gate="1" pin="A"/>
-<wire x1="-58.42" y1="55.88" x2="-58.42" y2="53.34" width="0.1524" layer="91"/>
-<wire x1="-58.42" y1="53.34" x2="-50.8" y2="53.34" width="0.1524" layer="91"/>
-<wire x1="-50.8" y1="53.34" x2="-50.8" y2="55.88" width="0.1524" layer="91"/>
-<pinref part="X88" gate="-3" pin="S"/>
-<wire x1="-50.8" y1="55.88" x2="-43.18" y2="55.88" width="0.1524" layer="91"/>
-<pinref part="X88" gate="-4" pin="S"/>
-<wire x1="-43.18" y1="55.88" x2="-43.18" y2="53.34" width="0.1524" layer="91"/>
-</segment>
-</net>
-<net name="N$17" class="0">
-<segment>
-<pinref part="R13" gate="G$1" pin="2"/>
-<pinref part="Q3" gate="1" pin="B"/>
-</segment>
-</net>
-<net name="N$19" class="0">
-<segment>
-<pinref part="Q3" gate="1" pin="C"/>
-<wire x1="-73.66" y1="66.04" x2="-58.42" y2="66.04" width="0.1524" layer="91"/>
-<wire x1="-58.42" y1="66.04" x2="-50.8" y2="66.04" width="0.1524" layer="91"/>
-<wire x1="-50.8" y1="66.04" x2="-50.8" y2="58.42" width="0.1524" layer="91"/>
-<pinref part="D4" gate="1" pin="C"/>
-<wire x1="-58.42" y1="60.96" x2="-58.42" y2="66.04" width="0.1524" layer="91"/>
-<pinref part="X88" gate="-2" pin="S"/>
-<wire x1="-50.8" y1="58.42" x2="-43.18" y2="58.42" width="0.1524" layer="91"/>
-<pinref part="X88" gate="-1" pin="S"/>
-<wire x1="-43.18" y1="60.96" x2="-43.18" y2="58.42" width="0.1524" layer="91"/>
+<pinref part="X77" gate="-3" pin="S"/>
+<pinref part="X77" gate="-4" pin="S"/>
+<wire x1="-49.53" y1="81.28" x2="-49.53" y2="78.74" width="0.1524" layer="91"/>
 </segment>
 </net>
@@
 <label x="-81.28" y="127" size="1.778" layer="95"/>
 </segment>
-<segment>
-<pinref part="R13" gate="G$1" pin="1"/>
-<wire x1="-88.9" y1="60.96" x2="-91.44" y2="60.96" width="0.1524" layer="91"/>
-<label x="-91.44" y="60.96" size="1.778" layer="95"/>
-</segment>
 </net>
 <net name="D8" class="0">
@@
 </segment>
 </net>
+<net name="D10" class="0">
+<segment>
+<pinref part="U$1" gate="G$1" pin="SDA"/>
+<wire x1="-147.32" y1="34.29" x2="-152.4" y2="34.29" width="0.1524" layer="91"/>
+<label x="-154.94" y="34.29" size="1.778" layer="95"/>
+</segment>
+</net>
+<net name="D11" class="0">
+<segment>
+<pinref part="U$1" gate="G$1" pin="SCK"/>
+<wire x1="-147.32" y1="36.83" x2="-152.4" y2="36.83" width="0.1524" layer="91"/>
+<label x="-154.94" y="36.83" size="1.778" layer="95"/>
+</segment>
+</net>
