File: KKK_valdiklis.sch (EAGLE design)
At the start: 65 parts, among them IC1 MCP1702-3.3, IC2 L293D, IC3 MCP1702-5.0, IC4 ATMEGA1284, IC5 DS1307, K1 S202T02, K2 S202T02, K3 S202T02, K4 S202T02, K5 S202T02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

Commit message: projektavimas
Parts:
- removed R16, R17: 330, resistor-1:R-US_0207/10
- added R1: 330, resistor-1:R-US_0207/10
- added R10: 1k, SteveMarple:RESISTOR
- added R13: 2.2k, adafruit:R-US_0207/10
- BAT1: value CR2032 -> (none); device SparkFun:BATTERY20PTH -> SparkFun-Electromechanical:BATTERY20PTH
- R15: value 2.2k -> 4.7K
- R2: value 1k -> 330; device SteveMarple:RESISTOR -> resistor-1:R-US_0207/10
- R6: value 10k -> 330; device SteveMarple:RESISTOR -> resistor-1:R-US_0207/10
- R7: value 330 -> 10k; device resistor-1:R-US_0207/10 -> SteveMarple:RESISTOR
- renumbered D1 to DIODE1, D3 to DIODE2
Connections:
- net !RESET: now also R7.1; no longer R6.1
- net D0: now also R1.1; no longer R7.1
- net D1: now also R2.1; no longer R4.1
- net D17(SDA): now also R13.1; no longer R15.1
- net D2: now also R15.2
- net D3: now also R4.1; no longer R5.1
- net D4: now also R5.1; no longer R17.1
- net D5: now also R6.1; no longer R16.1
- net N$24: now also R2.2; no longer R4.2
- net N$28: now also R4.2; no longer R5.2
- net N$31: now also R1.2; no longer R7.2
- net N$34: now also R6.2; no longer R16.2
- net N$37: now also R5.2; no longer R17.2
- net N$8: now also R10.1; no longer R2.1
- net VCC: now also R10.2, R13.2, R15.1, R7.2; no longer R15.2, R2.2, R6.2
Other:
- moved on the sheet: R15, R4, R5, X10-3

Commit message: projektavimas
Parts:
- removed C1, C2, C8: 1u, SparkFun:CAPPTH1
- removed IC1: MCP1702-3.3, burr-brown:REG1117
- removed IC3: MCP1702-5.0, burr-brown:REG1117
- removed JP5: 3V3/5V, SparkFun:JUMPER-3PTH
- removed JP6: VREG PWR, SparkFun:JUMPER-2PTH
Connections:
- removed net +5V: C1.1, IC1.VIN, JP5.3, JP6.2
- removed net D10: U$1.SDA
- removed net D102(RX1): IC4.PCINT26/INT0_PD2
- removed net D11: U$1.SCK
- removed net D6: IC2.1A, R12.1
- removed net D7: IC2.2A
- removed net D8: IC2.4A
- removed net D9: IC2.3A
- removed net N$14: IC3.VOUT, JP6.1
- removed net VIN: C8.1, IC3.VIN
- new net D10(RX1): IC2.2A, IC4.PCINT26/INT0_PD2
- net +3V3: no longer C2.1, IC1.VOUT, JP5.1
- net D11(TX1): now also IC2.1A
- net D12: now also IC2.3A; no longer U$1.LED
- net D13: now also IC2.4A; no longer U$1.A0
- net D14: now also R12.1; no longer U$1.RST
- net D15: now also U$1.LED; no longer U$1.CS
- net D18(TCK): now also U$1.SCK
- net D19(TMS): now also U$1.SDA
- net D20(TDO): now also U$1.A0
- net D21: now also U$1.RST
- net D22: now also U$1.CS
- net GND: no longer C1.2, C2.2, C8.2, IC1.GND, IC3.GND
- net VCC: no longer JP5.2
Other:
- note removed: "3V3 regulator"
- note removed: "5V regulator"
- note removed: "Power and connectors"

Commit message: projektavimas
Parts:
- X10: value (none) -> 22-23-2031; device con-phoenix-254:MPT3 -> con-molex:22-23-2031
Connections:
- net D2: no longer R15.2, X10-2.1
- net D6(MISO): now also R15.2, X10-2.S
- net GND: now also X10-1.S; no longer X10-1.1
- net VCC: now also X10-3.S; no longer X10-3.1
Changed lines of the file:
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@@
 <part name="P+19" library="supply1" deviceset="VCC" device=""/>
 <part name="C3" library="SparkFun" deviceset="CAP" device="PTH" value="100n"/>
-<part name="X10" library="con-phoenix-254" deviceset="MPT3" device=""/>
+<part name="X10" library="con-molex" deviceset="22-23-2031" device=""/>
 <part name="U$1" library="tft_1.8_1.44_oled_0.96" deviceset="1.8&quot;_TFT" device=""/>
 <part name="K4" library="relay-1" deviceset="S202T02" device=""/>
@@
 </segment>
 <segment>
-<pinref part="X10" gate="-1" pin="1"/>
+<pinref part="X10" gate="-1" pin="S"/>
 <wire x1="-27.94" y1="-44.45" x2="-35.56" y2="-44.45" width="0.1524" layer="91"/>
 <label x="-35.56" y="-44.45" size="1.778" layer="95"/>
@@
 </segment>
 <segment>
-<pinref part="X10" gate="-3" pin="1"/>
+<pinref part="X10" gate="-3" pin="S"/>
 <wire x1="-27.94" y1="-59.69" x2="-30.48" y2="-59.69" width="0.1524" layer="91"/>
 <pinref part="P+9" gate="VCC" pin="VCC"/>
@@
 <pinref part="IC4" gate="G$1" pin="PCINT14/MISO_PB6"/>
 </segment>
+<segment>
+<pinref part="X10" gate="-2" pin="S"/>
+<wire x1="-27.94" y1="-49.53" x2="-30.48" y2="-49.53" width="0.1524" layer="91"/>
+<label x="-44.45" y="-49.53" size="1.778" layer="95"/>
+<pinref part="R15" gate="G$1" pin="2"/>
+<wire x1="-30.48" y1="-49.53" x2="-44.45" y2="-49.53" width="0.1524" layer="91"/>
+<junction x="-30.48" y="-49.53"/>
+</segment>
 </net>
 <net name="D11(TX1)" class="0">
@@
 <net name="D2" class="0">
 <segment>
-<pinref part="X10" gate="-2" pin="1"/>
-<wire x1="-27.94" y1="-49.53" x2="-30.48" y2="-49.53" width="0.1524" layer="91"/>
-<label x="-35.56" y="-49.53" size="1.778" layer="95"/>
-<pinref part="R15" gate="G$1" pin="2"/>
-<wire x1="-30.48" y1="-49.53" x2="-35.56" y2="-49.53" width="0.1524" layer="91"/>
-<junction x="-30.48" y="-49.53"/>
-</segment>
-<segment>
 <wire x1="-7.62" y1="27.94" x2="-15.24" y2="27.94" width="0.1524" layer="91"/>

Commit message: trasavimas
Connections:
- net N$12 renamed D-
- net N$22 renamed D+
Changed lines of the file:
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@@
 <clearance class="1" value="0.2032"/>
 </class>
-<class number="3" name="antenna" width="0.6096" drill="0">
+<class number="2" name="D-" width="0" drill="0">
+</class>
+<class number="3" name="D+" width="0" drill="0">
 </class>
 <class number="5" name="220v" width="1" drill="0">
@@
 </segment>
 </net>
-<net name="N$12" class="0">
+<net name="D-" class="0">
 <segment>
 <pinref part="USB" gate="G$1" pin="D-"/>
@@
 </segment>
 </net>
-<net name="N$22" class="0">
+<net name="D+" class="0">
 <segment>
 <pinref part="U$2" gate="G$1" pin="UD+"/>
