File: KKK_valdiklis.sch (EAGLE design)
At the start: 56 parts, among them IC2 L293D, IC4 ATMEGA1284, IC5 DS1307, K1 S202T02, K2 S202T02, K3 S202T02, K4 S202T02, K5 S202T02, K6 S202T02, Q2 TIP120V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

Commit message: trasavimas
Parts:
- added AC-DC-5V: HLK-PM01_AC_DC, HLK-PM01:HLK-PM01_AC_DC
- added C2: (no value), rcl-1:C-EU025-024X044
- added J4: HEAD3X2, MyCON2:HEAD3X2
- added JP2: M02PTH2, SparkFun-Connectors-1:M02PTH2
- added U$4: 2-3.50, con-phoenix-350-1:2-3.50
Connections:
- removed net +3V3: U$1.3.3V
- removed net D5: IC4.PCINT13/MOSI_PB5, R6.1
- new net 220V: AC-DC-5V.AC1, U$4-1.K
- new net D5(MOSI): IC4.PCINT13/MOSI_PB5, J4.4, R6.1
- new net N$3: AC-DC-5V.AC0, JP2.1
- new net N$4: JP2.2, U$4-2.K
- net !RESET: now also J4.5
- net A0: no longer R11.1, R9.2, S2.S, S2.S1
- net A2: now also U$1.CS
- net A3: now also U$1.RST
- net A4: now also U$1.A0
- net A5: now also U$1.SDA
- net A6: now also U$1.SCK
- net A7: now also R11.1, R9.2, S2.S, S2.S1
- net D18(TCK): no longer U$1.SCK
- net D19(TMS): no longer U$1.SDA
- net D20(TDO): no longer U$1.A0
- net D21: no longer U$1.RST
- net D22: no longer U$1.CS
- net D6(MISO): now also J4.1
- net D7(SCK): now also J4.3
- net GND: now also AC-DC-5V.-V, C2.2, J4.6
- net VCC: now also AC-DC-5V.+V, C2.1, J4.2, U$1.3.3V
Other:
- note added: "ICSP"

Commit message: trasavimas
Connections:
- net D8(RX0): now also JP1.3; no longer JP1.2
- net D9(TX0): now also JP1.2; no longer JP1.3
- net GND: now also JP1.1
- net VCC: now also IC2.1-2EN, IC2.3-4EN
Changed lines of the file:
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@@
 <part name="GND6" library="supply1" deviceset="GND" device=""/>
 <part name="P+7" library="supply1" deviceset="VCC" device=""/>
+<part name="GND11" library="supply1" deviceset="GND" device=""/>
+<part name="P+8" library="supply1" deviceset="VCC" device=""/>
+<part name="P+12" library="supply1" deviceset="VCC" device=""/>
 </parts>
 <sheets>
@@
 <instance part="GND6" gate="1" x="91.44" y="154.94" rot="R270"/>
 <instance part="P+7" gate="VCC" x="-154.94" y="21.59" rot="R90"/>
+<instance part="GND11" gate="1" x="-92.71" y="-17.78" rot="R180"/>
+<instance part="P+8" gate="VCC" x="-35.56" y="119.38" rot="R270"/>
+<instance part="P+12" gate="VCC" x="-85.09" y="154.94" rot="R90"/>
 </instances>
 <busses>
@@
 <pinref part="GND6" gate="1" pin="GND"/>
 </segment>
+<segment>
+<pinref part="JP1" gate="G$1" pin="1"/>
+<pinref part="GND11" gate="1" pin="GND"/>
+<wire x1="-92.71" y1="-20.32" x2="-86.36" y2="-20.32" width="0.1524" layer="91"/>
+</segment>
 </net>
 <net name="VCC" class="1">
@@
 <junction x="-147.32" y="21.59"/>
 <pinref part="P+7" gate="VCC" pin="VCC"/>
+</segment>
+<segment>
+<pinref part="IC2" gate="G$1" pin="3-4EN"/>
+<pinref part="P+8" gate="VCC" pin="VCC"/>
+<wire x1="-38.1" y1="119.38" x2="-43.18" y2="119.38" width="0.1524" layer="91"/>
+</segment>
+<segment>
+<pinref part="IC2" gate="G$1" pin="1-2EN"/>
+<pinref part="P+12" gate="VCC" pin="VCC"/>
+<wire x1="-82.55" y1="154.94" x2="-73.66" y2="154.94" width="0.1524" layer="91"/>
 </segment>
 </net>
@@
 </segment>
 <segment>
-<wire x1="-86.36" y1="-25.4" x2="-87.63" y2="-25.4" width="0.1524" layer="91"/>
-<pinref part="JP1" gate="G$1" pin="3"/>
-<junction x="-86.36" y="-25.4"/>
-<label x="-87.63" y="-25.4" size="1.27" layer="95" rot="R180" xref="yes"/>
-</segment>
-</net>
-<net name="D8(RX0)" class="0">
-<segment>
-<wire x1="-7.62" y1="0" x2="-15.24" y2="0" width="0.1524" layer="91"/>
-<label x="-17.78" y="0" size="1.778" layer="95" rot="MR0"/>
-<pinref part="IC4" gate="G$1" pin="PCINT24/RXD0_PD0"/>
-</segment>
-<segment>
 <wire x1="-87.63" y1="-22.86" x2="-86.36" y2="-22.86" width="0.1524" layer="91"/>
 <wire x1="-86.36" y1="-22.86" x2="-87.63" y2="-22.86" width="0.1524" layer="91"/>
@@
 </segment>
 </net>
+<net name="D8(RX0)" class="0">
+<segment>
+<wire x1="-7.62" y1="0" x2="-15.24" y2="0" width="0.1524" layer="91"/>
+<label x="-17.78" y="0" size="1.778" layer="95" rot="MR0"/>
+<pinref part="IC4" gate="G$1" pin="PCINT24/RXD0_PD0"/>
+</segment>
+<segment>
+<wire x1="-86.36" y1="-25.4" x2="-87.63" y2="-25.4" width="0.1524" layer="91"/>
+<pinref part="JP1" gate="G$1" pin="3"/>
+<junction x="-86.36" y="-25.4"/>
+<label x="-87.63" y="-25.4" size="1.27" layer="95" rot="R180" xref="yes"/>
+</segment>
+</net>

Commit message: trasavimas
Parts:
- added X11: +12V, con-molex:22-23-2021
Connections:
- removed net +12V: IC2.VCC2
- new net N$5: IC2.VCC2, X11-2.S
- net D10(RX1): now also IC2.3A; no longer IC2.2A
- net D12: now also IC2.2A; no longer IC2.3A
- net GND: now also X11-1.S
Other:
- moved on the sheet: X7-1, X7-2, X8-1, X8-2
Changed lines of the file:
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@@
 <part name="GND15" library="SparkFun-Aesthetics" deviceset="GND" device=""/>
 <part name="GND18" library="SparkFun-Aesthetics" deviceset="GND" device=""/>
-<part name="SUPPLY1" library="supply2" deviceset="+12V" device=""/>
 <part name="X6" library="con-molex" deviceset="22-23-2021" device="" value="Floor heating"/>
 <part name="X1" library="con-molex" deviceset="22-23-2021" device="" value="Boiler pump"/>
@@
 <part name="P+8" library="supply1" deviceset="VCC" device=""/>
 <part name="P+12" library="supply1" deviceset="VCC" device=""/>
+<part name="X11" library="con-molex" deviceset="22-23-2021" device="" value="+12V"/>
+<part name="GND14" library="SparkFun-Aesthetics" deviceset="GND" device=""/>
 </parts>
 <sheets>
@@
 <instance part="GND15" gate="1" x="-38.1" y="137.16" rot="R90"/>
 <instance part="GND18" gate="1" x="-78.74" y="137.16" rot="R270"/>
-<instance part="SUPPLY1" gate="+12V" x="-76.2" y="119.38" rot="R90"/>
 <instance part="X6" gate="-1" x="25.4" y="78.74" smashed="yes">
 <attribute name="NAME" x="27.94" y="77.978" size="1.524" layer="95"/>
@@
 </instance>
 <instance part="X5" gate="-2" x="25.4" y="91.44"/>
-<instance part="X7" gate="-1" x="-73.66" y="106.68" smashed="yes">
-<attribute name="NAME" x="-71.12" y="105.918" size="1.524" layer="95"/>
-<attribute name="VALUE" x="-84.582" y="110.617" size="1.778" layer="96"/>
-</instance>
-<instance part="X7" gate="-2" x="-73.66" y="102.87"/>
-<instance part="X8" gate="-1" x="-44.45" y="106.68" smashed="yes">
-<attribute name="NAME" x="-41.91" y="105.918" size="1.524" layer="95"/>
-<attribute name="VALUE" x="-55.372" y="110.617" size="1.778" layer="96"/>
-</instance>
-<instance part="X8" gate="-2" x="-44.45" y="102.87"/>
+<instance part="X7" gate="-1" x="-74.93" y="102.87" smashed="yes">
+<attribute name="NAME" x="-72.39" y="102.108" size="1.524" layer="95"/>
+<attribute name="VALUE" x="-85.852" y="106.807" size="1.778" layer="96"/>
+</instance>
+<instance part="X7" gate="-2" x="-74.93" y="99.06"/>
+<instance part="X8" gate="-1" x="-45.72" y="102.87" smashed="yes">
+<attribute name="NAME" x="-43.18" y="102.108" size="1.524" layer="95"/>
+<attribute name="VALUE" x="-56.642" y="106.807" size="1.778" layer="96"/>
+</instance>
+<instance part="X8" gate="-2" x="-45.72" y="99.06"/>
 <instance part="GND3" gate="1" x="-160.02" y="21.59"/>
 <instance part="P+9" gate="VCC" x="-38.1" y="-59.69" rot="R90"/>
@@
 <instance part="P+7" gate="VCC" x="-154.94" y="21.59" rot="R90"/>
 <instance part="GND11" gate="1" x="-92.71" y="-17.78" rot="R180"/>
-<instance part="P+8" gate="VCC" x="-35.56" y="119.38" rot="R270"/>
-<instance part="P+12" gate="VCC" x="-85.09" y="154.94" rot="R90"/>
+<instance part="P+8" gate="VCC" x="-35.56" y="119.38" smashed="yes" rot="R270">
+<attribute name="VALUE" x="-38.1" y="120.65" size="1.778" layer="96"/>
+</instance>
+<instance part="P+12" gate="VCC" x="-85.09" y="154.94" smashed="yes" rot="R90">
+<attribute name="VALUE" x="-81.28" y="158.75" size="1.778" layer="96" rot="R180"/>
+</instance>
+<instance part="X11" gate="-1" x="-86.36" y="116.84" smashed="yes" rot="R180">
+<attribute name="NAME" x="-88.9" y="117.602" size="1.524" layer="95" rot="R180"/>
+<attribute name="VALUE" x="-89.408" y="123.063" size="1.778" layer="96" rot="R180"/>
+</instance>
+<instance part="X11" gate="-2" x="-86.36" y="119.38" rot="R180"/>
+<instance part="GND14" gate="1" x="-77.47" y="114.3"/>
 </instances>
 <busses>
@@
 <wire x1="-92.71" y1="-20.32" x2="-86.36" y2="-20.32" width="0.1524" layer="91"/>
 </segment>
+<segment>
+<pinref part="GND14" gate="1" pin="GND"/>
+<pinref part="X11" gate="-1" pin="S"/>
+<wire x1="-77.47" y1="116.84" x2="-83.82" y2="116.84" width="0.2032" layer="91"/>
+</segment>
 </net>
 <net name="VCC" class="1">
@@
 <pinref part="IC2" gate="G$1" pin="1A"/>
 <wire x1="-73.66" y1="149.86" x2="-81.28" y2="149.86" width="0.1524" layer="91"/>
-<label x="-81.28" y="152.4" size="1.778" layer="95"/>
+<label x="-85.09" y="151.13" size="1.778" layer="95"/>
 </segment>
 </net>
@@
 </segment>
 <segment>
-<pinref part="IC2" gate="G$1" pin="2A"/>
-<wire x1="-73.66" y1="124.46" x2="-81.28" y2="124.46" width="0.1524" layer="91"/>
-<label x="-81.28" y="127" size="1.778" layer="95"/>
+<pinref part="IC2" gate="G$1" pin="3A"/>
+<wire x1="-43.18" y1="124.46" x2="-35.56" y2="124.46" width="0.1524" layer="91"/>
+<label x="-38.1" y="125.73" size="1.778" layer="95"/>
 </segment>
 </net>
@@
 </segment>
 <segment>
-<pinref part="IC2" gate="G$1" pin="3A"/>
-<wire x1="-43.18" y1="124.46" x2="-35.56" y2="124.46" width="0.1524" layer="91"/>
-<label x="-38.1" y="127" size="1.778" layer="95"/>
+<pinref part="IC2" gate="G$1" pin="2A"/>
+<wire x1="-73.66" y1="124.46" x2="-81.28" y2="124.46" width="0.1524" layer="91"/>
+<label x="-85.09" y="125.73" size="1.778" layer="95"/>
 </segment>
 </net>
@@
 <pinref part="IC2" gate="G$1" pin="4A"/>
 <wire x1="-43.18" y1="149.86" x2="-35.56" y2="149.86" width="0.1524" layer="91"/>
-<label x="-38.1" y="152.4" size="1.778" layer="95"/>
+<label x="-38.1" y="151.13" size="1.778" layer="95"/>
 </segment>
 </net>
@@
 </segment>
 </net>
-<net name="+12V" class="0">
-<segment>
-<pinref part="IC2" gate="G$1" pin="VCC2"/>
-<pinref part="SUPPLY1" gate="+12V" pin="+12V"/>
-</segment>
-</net>
 <net name="MV1.1" class="0">
 <segment>
 <pinref part="IC2" gate="G$1" pin="1Y"/>
 <wire x1="-73.66" y1="144.78" x2="-81.28" y2="144.78" width="0.1524" layer="91"/>
-<label x="-83.82" y="147.32" size="1.778" layer="95"/>
+<label x="-85.09" y="146.05" size="1.778" layer="95"/>
 </segment>
 <segment>
 <pinref part="X7" gate="-1" pin="S"/>
-<wire x1="-76.2" y1="106.68" x2="-81.28" y2="106.68" width="0.1524" layer="91"/>
-<label x="-81.28" y="107.95" size="1.778" layer="95"/>
+<wire x1="-77.47" y1="102.87" x2="-82.55" y2="102.87" width="0.1524" layer="91"/>
+<label x="-82.55" y="104.14" size="1.778" layer="95"/>
 </segment>
 </net>
@@
 <pinref part="IC2" gate="G$1" pin="2Y"/>
 <wire x1="-73.66" y1="129.54" x2="-81.28" y2="129.54" width="0.1524" layer="91"/>
-<label x="-83.82" y="132.08" size="1.778" layer="95"/>
+<label x="-85.09" y="130.81" size="1.778" layer="95"/>
 </segment>
 <segment>
 <pinref part="X7" gate="-2" pin="S"/>
-<wire x1="-76.2" y1="102.87" x2="-81.28" y2="102.87" width="0.1524" layer="91"/>
-<label x="-81.28" y="104.14" size="1.778" layer="95"/>
+<wire x1="-77.47" y1="99.06" x2="-82.55" y2="99.06" width="0.1524" layer="91"/>
+<label x="-82.55" y="100.33" size="1.778" layer="95"/>
 </segment>
 </net>
@@
 <pinref part="IC2" gate="G$1" pin="4Y"/>
 <wire x1="-43.18" y1="144.78" x2="-35.56" y2="144.78" width="0.1524" layer="91"/>
-<label x="-35.56" y="147.32" size="1.778" layer="95"/>
+<label x="-38.1" y="146.05" size="1.778" layer="95"/>
 </segment>
 <segment>
 <pinref part="X8" gate="-1" pin="S"/>
-<wire x1="-46.99" y1="106.68" x2="-52.07" y2="106.68" width="0.1524" layer="91"/>
-<label x="-52.07" y="107.95" size="1.778" layer="95"/>
+<wire x1="-48.26" y1="102.87" x2="-53.34" y2="102.87" width="0.1524" layer="91"/>
+<label x="-53.34" y="104.14" size="1.778" layer="95"/>
 </segment>
 </net>
@@
 <pinref part="IC2" gate="G$1" pin="3Y"/>
 <wire x1="-43.18" y1="129.54" x2="-35.56" y2="129.54" width="0.1524" layer="91"/>
-<label x="-35.56" y="132.08" size="1.778" layer="95"/>
+<label x="-38.1" y="130.81" size="1.778" layer="95"/>
 </segment>
 <segment>
 <pinref part="X8" gate="-2" pin="S"/>
-<wire x1="-46.99" y1="102.87" x2="-52.07" y2="102.87" width="0.1524" layer="91"/>
-<label x="-52.07" y="104.14" size="1.778" layer="95"/>
+<wire x1="-48.26" y1="99.06" x2="-53.34" y2="99.06" width="0.1524" layer="91"/>
+<label x="-53.34" y="100.33" size="1.778" layer="95"/>
 </segment>
 </net>
@@
 </segment>
 </net>
+<net name="N$5" class="0">
+<segment>
+<pinref part="IC2" gate="G$1" pin="VCC2"/>
+<pinref part="X11" gate="-2" pin="S"/>
+<wire x1="-73.66" y1="119.38" x2="-83.82" y2="119.38" width="0.2032" layer="91"/>
+</segment>
+</net>

Commit message: trasavimas
Parts:
- renumbered Q2 to T2
Connections:
- removed net N$5: IC2.VCC2, X11-2.S
- new net +12V: IC2.VCC2, X11-2.S, X77-4.S
- net N$15: no longer X77-4.S
Other:
- moved on the sheet: DIODE2, X77-1, X77-2, X77-4
Changed lines of the file:
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@@
 <part name="R9" library="resistor" deviceset="R-EU_" device="0207/10" value="1k"/>
 <part name="R11" library="resistor" deviceset="R-EU_" device="0207/10" value="2k"/>
-<part name="Q2" library="rocketfarm" deviceset="TIP120" device="V"/>
+<part name="T2" library="rocketfarm" deviceset="TIP120" device="V"/>
 <part name="X77" library="con-molex" deviceset="22-23-2041" device="" value="PUMP1"/>
 <part name="R12" library="resistor" deviceset="R-EU_" device="0207/10" value="2k"/>
@@
 <part name="X11" library="con-molex" deviceset="22-23-2021" device="" value="+12V"/>
 <part name="GND14" library="SparkFun-Aesthetics" deviceset="GND" device=""/>
+<part name="GND19" library="SparkFun-Aesthetics" deviceset="GND" device=""/>
 </parts>
 <sheets>
@@
 <instance part="R9" gate="G$1" x="175.26" y="7.62" rot="R90"/>
 <instance part="R11" gate="G$1" x="175.26" y="22.86" rot="R90"/>
-<instance part="Q2" gate="1" x="-76.2" y="76.2"/>
-<instance part="X77" gate="-1" x="-46.99" y="71.12"/>
-<instance part="X77" gate="-2" x="-46.99" y="68.58"/>
+<instance part="T2" gate="1" x="-76.2" y="76.2" smashed="yes">
+<attribute name="NAME" x="-78.74" y="80.01" size="1.778" layer="95"/>
+<attribute name="VALUE" x="-78.74" y="82.55" size="1.778" layer="96"/>
+</instance>
+<instance part="X77" gate="-1" x="-46.99" y="72.39"/>
+<instance part="X77" gate="-2" x="-46.99" y="69.85"/>
 <instance part="X77" gate="-3" x="-46.99" y="81.28"/>
-<instance part="X77" gate="-4" x="-46.99" y="78.74"/>
+<instance part="X77" gate="-4" x="-46.99" y="83.82"/>
 <instance part="R12" gate="G$1" x="-83.82" y="76.2" smashed="yes">
 <attribute name="NAME" x="-87.63" y="77.6986" size="1.778" layer="95"/>
 <attribute name="VALUE" x="-82.55" y="77.978" size="1.778" layer="96"/>
 </instance>
-<instance part="DIODE2" gate="1" x="-58.42" y="73.66" rot="R90"/>
+<instance part="DIODE2" gate="1" x="-58.42" y="74.93" smashed="yes" rot="R90">
+<attribute name="NAME" x="-69.85" y="79.2226" size="1.778" layer="95"/>
+<attribute name="VALUE" x="-69.85" y="76.4286" size="1.778" layer="96"/>
+</instance>
 <instance part="Q4" gate="G$1" x="142.24" y="91.44" rot="R180"/>
 <instance part="IC5" gate="G$1" x="144.78" y="68.58"/>
@@
 <instance part="X11" gate="-2" x="-86.36" y="119.38" rot="R180"/>
 <instance part="GND14" gate="1" x="-77.47" y="114.3"/>
+<instance part="GND19" gate="1" x="-58.42" y="67.31"/>
 </instances>
 <busses>
@@
 </segment>
 <segment>
-<pinref part="Q2" gate="1" pin="E"/>
-<wire x1="-73.66" y1="71.12" x2="-73.66" y2="68.58" width="0.1524" layer="91"/>
-<wire x1="-73.66" y1="68.58" x2="-58.42" y2="68.58" width="0.1524" layer="91"/>
+<pinref part="T2" gate="1" pin="E"/>
+<wire x1="-73.66" y1="71.12" x2="-73.66" y2="69.85" width="0.1524" layer="91"/>
+<wire x1="-73.66" y1="69.85" x2="-58.42" y2="69.85" width="0.1524" layer="91"/>
 <pinref part="DIODE2" gate="1" pin="A"/>
-<wire x1="-58.42" y1="71.12" x2="-58.42" y2="68.58" width="0.1524" layer="91"/>
-<wire x1="-58.42" y1="68.58" x2="-49.53" y2="68.58" width="0.1524" layer="91"/>
+<wire x1="-58.42" y1="72.39" x2="-58.42" y2="69.85" width="0.1524" layer="91"/>
+<wire x1="-58.42" y1="69.85" x2="-49.53" y2="69.85" width="0.1524" layer="91"/>
 <pinref part="X77" gate="-2" pin="S"/>
 <pinref part="X77" gate="-1" pin="S"/>
-<wire x1="-49.53" y1="68.58" x2="-49.53" y2="71.12" width="0.1524" layer="91"/>
+<wire x1="-49.53" y1="69.85" x2="-49.53" y2="72.39" width="0.1524" layer="91"/>
+<pinref part="GND19" gate="1" pin="GND"/>
+<junction x="-58.42" y="69.85"/>
 </segment>
 <segment>
@@
 <segment>
 <pinref part="R12" gate="G$1" pin="2"/>
-<pinref part="Q2" gate="1" pin="B"/>
+<pinref part="T2" gate="1" pin="B"/>
 </segment>
 </net>
 <net name="N$15" class="0">
 <segment>
-<pinref part="Q2" gate="1" pin="C"/>
+<pinref part="T2" gate="1" pin="C"/>
 <wire x1="-73.66" y1="81.28" x2="-58.42" y2="81.28" width="0.1524" layer="91"/>
 <wire x1="-58.42" y1="81.28" x2="-49.53" y2="81.28" width="0.1524" layer="91"/>
 <pinref part="DIODE2" gate="1" pin="C"/>
-<wire x1="-58.42" y1="76.2" x2="-58.42" y2="81.28" width="0.1524" layer="91"/>
+<wire x1="-58.42" y1="77.47" x2="-58.42" y2="81.28" width="0.1524" layer="91"/>
 <pinref part="X77" gate="-3" pin="S"/>
-<pinref part="X77" gate="-4" pin="S"/>
-<wire x1="-49.53" y1="81.28" x2="-49.53" y2="78.74" width="0.1524" layer="91"/>
 </segment>
 </net>
@@
 </segment>
 </net>
-<net name="N$5" class="0">
+<net name="+12V" class="0">
+<segment>
+<pinref part="X77" gate="-4" pin="S"/>
+<wire x1="-49.53" y1="83.82" x2="-52.07" y2="83.82" width="0.2032" layer="91"/>
+<label x="-52.07" y="83.82" size="1.27" layer="95" rot="R180" xref="yes"/>
+</segment>
 <segment>
 <pinref part="IC2" gate="G$1" pin="VCC2"/>
