File: KKK_valdiklis.job.brd (EAGLE design)
At the start: 120 x 100 mm, 67 parts, among them IC2 L293D, IC4 ATMEGA1284, IC5 DS1307, J4 HEAD3X2, K1 S202T02, K2 S202T02, K3 S202T02, K4 S202T02, K5 S202T02, K6 S202T02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

Commit message: trasavimas
Parts:
- removed C4: 100n, SparkFun:CAP-PTH-SMALL
- removed JP3: USB-B, SparkFun-Connectors-1:USB-B-PTH
- added C17: 0.1uF, rcl:C0805K
- added USB1: USB-B-H, con-usb-2:USB-B-H
- moved BAT1 15.3 mm to (109.2, 80.0), turned to 270 degrees
- moved C3 2.84 mm to (3.81, 82.5)
- moved U$2 1.27 mm to (7.62, 88.9)
- moved Y1 1.27 mm to (15.2, 77.5)
Connections:
- net !RESET: now also C17.2; no longer C4.1
- net +5V: now also USB1.VBUS; no longer JP3.VBUS
- net GND: now also USB1.GND, USB1.GND@1; no longer JP3.GND
- net N$11: now also C17.1; no longer C4.2
- net N$12: now also USB1.D+; no longer JP3.D-
- net N$22: now also USB1.D-; no longer JP3.D+
Routing:
- net !RESET: track 146.7 -> 165.7 mm, vias 2 -> 1
- net GND: track 487.7 -> 506.7 mm
- net N$27: track 28.6 -> 15.0 mm
- net +5V: track 22.8 -> 27.3 mm
- net N$12: track 14.5 -> 16.9 mm, vias 1 -> 0
- net N$22: track 14.8 -> 12.5 mm, vias 1 -> 0
- net N$11: track 4.34 -> 6.35 mm
- net N$9: track 5.61 -> 7.40 mm, vias 0 -> 1
- net N$7: track 14.8 -> 13.0 mm, vias 0 -> 2
- net N$14: track 5.08 -> 3.81 mm
