File: 3K_valdiklis_v1/3K_valdiklis_v1.brd (EAGLE design)
At the start: 120 x 100 mm, 67 parts, among them IC2 L293D, IC4 ATMEGA1284, IC5 DS1307, J4 HEAD3X2, K1 S202T02, K2 S202T02, K3 S202T02, K4 S202T02, K5 S202T02, K6 S202T02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

Commit message: trasavimas
Parts:
- removed C17: 0.1uF, rcl:C0805K
- removed JP1: (no value), SparkFun-Connectors-1:1X05
- removed USB1: USB-B-H, con-usb-2:USB-B-H
- added C4: 100n, SparkFun:CAP-PTH-SMALL
- added JP3: USB-B, SparkFun-Connectors-1:USB-B-PTH
- moved BAT1 15.3 mm to (97.8, 69.8), turned to 0 degrees
- moved J4 5.08 mm to (22.2, 50.2)
- moved U$2 1.27 mm to (8.89, 88.9)
- moved C3 1.27 mm to (3.81, 81.3)
- moved Y1 1.27 mm to (15.2, 78.7)
Connections:
- removed net 0(RX0): U$2.2
- removed net 1(TX0): U$2.3
- net !RESET: now also C4.1; no longer C17.2
- net +5V: now also JP3.VBUS; no longer USB1.VBUS
- net D8(RX0): now also U$2.3; no longer JP1.3
- net D9(TX0): now also U$2.2; no longer JP1.2
- net DTR: no longer JP1.4
- net GND: now also JP3.GND; no longer JP1.1, USB1.GND, USB1.GND@1
- net N$11: now also C4.2; no longer C17.1
- net N$12: now also JP3.D-; no longer USB1.D+
- net N$22: now also JP3.D+; no longer USB1.D-
Routing:
- net D9(TX0): track 73.0 -> 120.7 mm, vias 1 -> 4
- net GND: track 506.7 -> 461.7 mm
- net DTR: track 32.8 -> 0.00 mm, vias 1 -> 0
- net D8(RX0): track 61.3 -> 84.6 mm, vias 1 -> 4
- net !RESET: track 165.7 -> 147.1 mm, vias 1 -> 3
- net N$27: track 15.0 -> 28.6 mm
- net D5(MOSI): track 54.7 -> 61.7 mm, vias 0 -> 2
- net AVCC: track 83.4 -> 76.8 mm, vias 1 -> 0
- net D6(MISO): track 80.9 -> 85.8 mm, vias 0 -> 1
- net D7(SCK): track 27.1 -> 32.0 mm, vias 0 -> 1
- net +5V: track 27.3 -> 32.0 mm
- net VCC: track 264.9 -> 261.1 mm
- net N$22: track 12.5 -> 16.3 mm
- net N$11: track 6.35 -> 4.34 mm
- net N$14: track 3.81 -> 5.61 mm
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
Commit message: trasavimas
Parts:
- moved R11 3.24 mm to (87.6, 86.4)
Routing:
- net N$17: track 0.00 -> 170.1 mm, vias 0 -> 1
- net VCC: track 261.1 -> 267.1 mm
- net D16(SCL): track 24.2 -> 20.0 mm
- net A7: track 93.9 -> 95.5 mm
- net D10(RX1): track 67.1 -> 66.1 mm
- net N$37: track 6.02 -> 5.13 mm
- net GND: track 461.7 -> 462.4 mm
- net AREF: track 50.3 -> 49.7 mm
- net D12: track 39.1 -> 38.6 mm
- net D15: track 72.6 -> 72.2 mm, vias 0 -> 1
- net !RESET: track 147.1 -> 147.2 mm, vias 3 -> 2
- net D8(RX0): vias 4 -> 2
Other:
- outline, holes or cut-outs redrawn

Commit message: trasavimas
Routing:
- net N$17: track 170.1 -> 85.0 mm, vias 1 -> 0
- net N$38: track 0.00 -> 85.0 mm
- net GND: track 462.4 -> 468.7 mm, vias 0 -> 1
- net VCC: track 267.1 -> 264.3 mm
- net N$41: track 8.15 -> 8.12 mm, vias 0 -> 1
- net N$40: track 8.15 -> 8.12 mm, vias 0 -> 1
- net N$35: track 8.15 -> 8.12 mm, vias 0 -> 1
- net N$18: track 8.15 -> 8.12 mm, vias 0 -> 1
- net N$19: track 8.15 -> 8.12 mm, vias 0 -> 1

Commit message: trasavimas
be klaidų!!
Connections:
- removed net +5V: JP3.VBUS, U$2.16
- new net N$19: IC2.8, X11.2
- net +12V: no longer IC2.8, X11.2
- net VCC: now also JP3.VBUS, U$2.16
Routing:
- net N$17: track 85.0 -> 170.1 mm, vias 0 -> 1
- net N$38 (its old number): track 85.0 -> 0.00 mm
- net VCC: track 264.3 -> 309.1 mm
- net +5V: track 32.0 -> 0.00 mm
- net GND: track 468.7 -> 452.8 mm, vias 1 -> 0
- net +12V: track 23.8 -> 12.8 mm
- net N$35: track 8.12 -> 8.15 mm, vias 1 -> 0
- net N$38: track 8.12 -> 8.15 mm, vias 1 -> 0
- net N$25: track 8.12 -> 8.15 mm, vias 1 -> 0
- net N$18: track 8.12 -> 8.15 mm, vias 1 -> 0
- net N$29: track 8.12 -> 8.15 mm, vias 1 -> 0
