File: 3K_valdiklis_v1/3K_valdiklis_v1.brd (EAGLE design)
At the start: 120 x 90 mm, 66 parts, among them IC2 L293D, IC4 ATMEGA1284, IC5 DS1307, J4 HEAD3X2, K1 S202T02, K2 S202T02, K3 S202T02, K4 S202T02, K5 S202T02, K6 S202T02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

Commit message: TRASAvimas
Parts:
- moved C3 1.80 mm to (6.35, 73.7)
- moved C13 1.27 mm to (30.5, 40.6), turned to 180 degrees
- moved U$2 1.27 mm to (10.2, 81.3)
- moved C4 1.27 mm to (10.2, 87.6)
Connections:
- removed net N$15: DIODE2.C, T2.C, X77.3
- net +12V: now also DIODE2.C, T2.C, X77.3
Routing:
- net N$17: track 170.1 -> 0.00 mm, vias 1 -> 0
- net XBOT: track 0.00 -> 85.0 mm
- net N$15: track 13.2 -> 68.0 mm
- net D8(RX0): track 90.8 -> 134.1 mm, vias 4 -> 2
- net D9(TX0): track 86.5 -> 105.5 mm, vias 4 -> 2
- net GND: track 491.9 -> 483.4 mm
- net +12V: track 12.8 -> 15.8 mm
- net N$14: track 3.81 -> 5.08 mm
- net N$11: track 2.54 -> 3.81 mm
- net !RESET: track 135.8 -> 137.1 mm
- net N$7: track 9.98 -> 9.46 mm
- net N$22: track 13.8 -> 14.3 mm
- net N$12: track 13.5 -> 14.0 mm
- net N$9: track 4.34 -> 3.81 mm
