File: 3K_valdiklis_v1/3K_valdiklis_v1.2.brd (EAGLE design)
At the start: 138 x 90 mm, 66 parts, among them IC2 L293D, IC4 ATMEGA1284, J4 HEAD3X2, K1 S202T02, K2 S202T02, K3 S202T02, K4 S202T02, K5 S202T02, K6 S202T02, T2 TIP120V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

Commit message: Trasavimas
Parts:
- moved U$3 4.95 mm to (123.3, 15.9)
- moved AC-DC-5V 4.95 mm to (23.0, 12.7)
- moved C10 4.95 mm to (61.1, 33.0)
- moved C11 4.95 mm to (57.9, 33.0)
- moved C2 4.95 mm to (50.9, 34.9)
- moved C3 4.95 mm to (86.5, 83.2)
- moved C4 4.95 mm to (99.8, 78.1)
- moved C5 4.95 mm to (89.5, 40.0)
- moved C6 4.95 mm to (106.2, 6.99)
- moved C7 4.95 mm to (129.0, 36.2)
- moved C9 4.95 mm to (39.4, 34.4)
- moved DIODE2 4.95 mm to (53.5, 69.7)
- moved IC2 4.95 mm to (38.2, 21.1)
- moved IC4 4.95 mm to (75.1, 36.8)
- moved JP12 4.95 mm to (43.9, 81.9)
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Routing:
- net D13: track 52.1 -> 38.0 mm
- net GND: track 450.1 -> 453.5 mm, vias 1 -> 3
