File: 3K_valdiklis_v1/3K_valdiklis_v1.2.job.brd (EAGLE design)
At the start: 120 x 90 mm, 66 parts, among them IC2 L293D, IC4 ATMEGA1284, IC5 DS1307, J4 HEAD3X2, K1 S202T02, K2 S202T02, K3 S202T02, K4 S202T02, K5 S202T02, K6 S202T02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

Commit message: TRASAvimas
Parts:
- removed BAT1: (no value), SparkFun-Electromechanical:BATTCOM_20MM_PTH
- removed C1: 22p, SparkFun:CAP-PTH-SMALL
- removed IC5: DS1307, adafruit:DIL08
- removed Q4: 32.768, crystal:TC38H
- removed R13: 2.2k, adafruit:0207/10
- removed R14: 2.2K, adafruit:0207/10
- added U$3: RTC-EEPROM-BATTERY, diy-modules-1:RTC_EEPROM_BATTERY
- moved U$1 135.2 mm to (146.7, 30.5), turned to 90 degrees
- moved X6 102.9 mm to (6.99, 87.6), turned to 0 degrees
- moved C4 100.0 mm to (109.9, 78.1), turned to 90 degrees
- moved X77 96.4 mm to (61.6, 86.9), turned to 0 degrees
- moved X5 95.1 mm to (14.6, 87.6), turned to 0 degrees
- moved U$2 94.0 mm to (102.9, 78.7), turned to 270 degrees
- moved C3 91.8 mm to (96.5, 83.2), turned to 270 degrees
- moved X4 89.4 mm to (22.2, 87.6), turned to 0 degrees
- moved X1 87.1 mm to (45.1, 87.6), turned to 0 degrees
- moved X3 85.9 mm to (29.8, 87.6), turned to 0 degrees
- moved X2 85.1 mm to (37.5, 87.6), turned to 0 degrees
- moved K6 83.1 mm to (6.99, 74.9), turned to 270 degrees
- moved T2 78.8 mm to (61.6, 77.3), turned to 180 degrees
- moved JP3 77.6 mm to (81.9, 82.5), turned to 270 degrees
- moved Y1 76.2 mm to (91.4, 72.4), turned to 0 degrees
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Connections:
- removed net DTR: C1.1
- removed net N$15: DIODE2.C, T2.C, X77.3
- removed net N$20: IC5.1, Q4.2
- removed net N$21: IC5.2, Q4.1
- removed net N$27: BAT1.1, IC5.3
- removed net SQW: IC5.7
- new net GND.2: U$3.J2.2
- new net N$17: U$3.J1.5
- new net VCC.2: U$3.J2.3
- net !RESET: no longer C1.2
- net +12V: now also DIODE2.C, T2.C, X77.3
- net D0: now also R12.1
- net D10(RX1): no longer IC2.10
- net D11(TX1): now also IC2.10; no longer IC2.2
- net D12: now also IC2.2; no longer IC2.7
- net D13: now also IC2.7; no longer IC2.15
- net D14: now also IC2.15; no longer R12.1
- net D16(SCL): now also U$3.J1.4; no longer IC5.6, R14.2
- net D17(SDA): now also U$3.J1.3; no longer IC5.5, R13.1
- net GND: now also U$3.J1.1; no longer BAT1.2, IC5.4
- net VCC: now also U$3.J1.2; no longer IC5.8, R13.2, R14.1
Routing:
- net N$17: track 170.1 -> 0.00 mm, vias 1 -> 0
- net D17(SDA): track 23.6 -> 97.5 mm
- net GND: track 510.6 -> 437.2 mm
- net D10(RX1): track 66.1 -> 0.00 mm
- net VCC: track 297.4 -> 361.1 mm, vias 0 -> 2
- net D12: track 38.6 -> 95.7 mm
- net D16(SCL): track 20.0 -> 73.0 mm
- net D4: track 19.1 -> 56.9 mm
- net AREF: track 44.6 -> 7.12 mm, vias 1 -> 0
- net D3: track 14.8 -> 48.5 mm
- net A2: track 25.7 -> 56.1 mm
- net D2: track 12.7 -> 39.8 mm
- net A3: track 25.7 -> 52.5 mm
- net N$20: track 3.81 -> 27.9 mm
- net A4: track 25.7 -> 48.4 mm
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Other:
- board size 120 x 90 mm -> 150 x 90 mm
