File: 3K_valdiklis_v1/3K_valdiklis_v1.sch (EAGLE design)
At the start: 67 parts, among them IC2 L293D, IC4 ATMEGA1284, IC5 DS1307, J4 HEAD3X2, K1 S202T02, K2 S202T02, K3 S202T02, K4 S202T02, K5 S202T02, K6 S202T02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

Commit message: trasavimas
Parts:
- removed C17: 0.1uF, rcl:C-USC0805K
- removed JP1: (no value), SparkFun-Connectors-1:M05PTH
- removed USB1: USB-B-H, con-usb-2:USB-B-H
- added C4: 100n, SparkFun:CAPPTH
- added JP3: USB-B, SparkFun-Connectors-1:USBPTH
Connections:
- removed net 0(RX0): U$2.TXD
- removed net 1(TX0): U$2.RXD
- net !RESET: now also C4.1; no longer C17.2
- net +5V: now also JP3.VBUS; no longer USB1.VBUS
- net D8(RX0): now also U$2.RXD; no longer JP1.3
- net D9(TX0): now also U$2.TXD; no longer JP1.2
- net DTR: no longer JP1.4
- net GND: now also JP3.GND; no longer JP1.1, USB1.GND, USB1.GND@1, USB1.GND@2
- net N$11: now also C4.2; no longer C17.1
- net N$12: now also JP3.D-; no longer USB1.D+
- net N$22: now also JP3.D+; no longer USB1.D-
Other:
- moved on the sheet: C3, Y1

Commit message: trasavimas
be klaidų!!
Connections:
- removed net +5V: JP3.VBUS, U$2.VCC
- new net N$19: IC2.VCC2, X11-2.S
- net +12V: no longer IC2.VCC2, X11-2.S
- net VCC: now also JP3.VBUS, U$2.VCC
Changed lines of the file:
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@@
 <setting verticaltext="up"/>
 </settings>
-<grid distance="0.1" unitdist="inch" unit="inch" style="lines" multiple="1" display="no" altdistance="0.01" altunitdist="inch" altunit="inch"/>
+<grid distance="0.127" unitdist="mm" unit="mm" style="lines" multiple="1" display="no" altdistance="0.01" altunitdist="inch" altunit="inch"/>
 <layers>
 <layer number="1" name="Top" color="4" fill="1" visible="no" active="no"/>
@@
 <part name="GND23" library="SparkFun" deviceset="GND" device=""/>
 <part name="U$2" library="ch340" deviceset="CH340G" device=""/>
-<part name="+3V9" library="supply1" deviceset="+5V" device=""/>
 <part name="Y1" library="SparkFun-FreqCtrl" deviceset="RESONATOR" device="PTH" value="12mhz"/>
 <part name="C3" library="SparkFun" deviceset="CAP" device="PTH" value="100n"/>
 <part name="C4" library="SparkFun" deviceset="CAP" device="PTH" value="100n"/>
 <part name="JP3" library="SparkFun-Connectors-1" deviceset="USB" device="PTH" value="USB-B"/>
+<part name="P+15" library="supply1" deviceset="VCC" device=""/>
 </parts>
 <sheets>
@@
 <instance part="GND23" gate="1" x="-162.56" y="125.984"/>
 <instance part="U$2" gate="G$1" x="-129.54" y="154.94"/>
-<instance part="+3V9" gate="1" x="-149.86" y="129.54" smashed="yes" rot="R90">
-<attribute name="VALUE" x="-148.59" y="128.27" size="1.778" layer="96" rot="R180"/>
-</instance>
 <instance part="Y1" gate="G$1" x="-152.4" y="144.78" smashed="yes" rot="R270">
 <attribute name="NAME" x="-151.384" y="142.24" size="1.778" layer="95" rot="R270"/>
@@
 </instance>
 <instance part="JP3" gate="G$1" x="-134.62" y="132.08" rot="MR180"/>
+<instance part="P+15" gate="VCC" x="-110.49" y="119.38" smashed="yes" rot="R270">
+<attribute name="VALUE" x="-114.3" y="115.57" size="1.778" layer="96"/>
+</instance>
 </instances>
 <busses>
@@
 <pinref part="C1" gate="G$1" pin="2"/>
 <wire x1="-96.52" y1="7.62" x2="-88.9" y2="7.62" width="0.2032" layer="91"/>
+<junction x="-88.9" y="7.62"/>
 </segment>
 <segment>
@@
 <pinref part="C10" gate="G$1" pin="2"/>
 <wire x1="-40.64" y1="-17.78" x2="-33.02" y2="-17.78" width="0.1524" layer="91"/>
+<junction x="-33.02" y="-17.78"/>
 </segment>
 <segment>
@@
 <pinref part="S1" gate="S" pin="2"/>
 <pinref part="GND1" gate="1" pin="GND"/>
+<junction x="-88.9" y="-2.54"/>
 </segment>
 <segment>
@@
 <pinref part="GND19" gate="1" pin="GND"/>
 <junction x="-58.42" y="69.85"/>
+<junction x="-49.53" y="69.85"/>
+<junction x="-49.53" y="72.39"/>
 </segment>
 <segment>
@@
 <wire x1="-73.66" y1="137.16" x2="-73.66" y2="134.62" width="0.1524" layer="91"/>
 <wire x1="-76.2" y1="137.16" x2="-73.66" y2="137.16" width="0.1524" layer="91"/>
+<junction x="-73.66" y="137.16"/>
 </segment>
 <segment>
@@
 <wire x1="-43.18" y1="137.16" x2="-43.18" y2="134.62" width="0.1524" layer="91"/>
 <wire x1="-40.64" y1="137.16" x2="-43.18" y2="137.16" width="0.1524" layer="91"/>
+<junction x="-43.18" y="137.16"/>
 </segment>
 <segment>
@@
 </segment>
 <segment>
-<wire x1="104.394" y1="154.94" x2="98.298" y2="154.94" width="0.1524" layer="91"/>
+<wire x1="104.394" y1="154.94" x2="98.425" y2="154.94" width="0.1524" layer="91"/>
+<wire x1="98.425" y1="154.94" x2="98.298" y2="154.94" width="0.1524" layer="91"/>
 <wire x1="98.298" y1="154.94" x2="93.98" y2="154.94" width="0.1524" layer="91"/>
 <pinref part="C2" gate="G$1" pin="2"/>
@@
 <wire x1="104.394" y1="154.94" x2="104.394" y2="157.48" width="0.1524" layer="91"/>
 <pinref part="GND6" gate="1" pin="GND"/>
+<junction x="98.425" y="154.94"/>
+<junction x="98.298" y="154.94"/>
 </segment>
 <segment>
@@
 <segment>
 <wire x1="93.98" y1="165.1" x2="98.298" y2="165.1" width="0.1524" layer="91"/>
-<wire x1="98.298" y1="165.1" x2="104.394" y2="165.1" width="0.1524" layer="91"/>
+<wire x1="98.298" y1="165.1" x2="98.425" y2="165.1" width="0.1524" layer="91"/>
 <pinref part="C2" gate="G$1" pin="1"/>
+<wire x1="98.425" y1="165.1" x2="104.394" y2="165.1" width="0.1524" layer="91"/>
 <wire x1="98.298" y1="163.83" x2="98.298" y2="165.1" width="0.1524" layer="91"/>
 <pinref part="AC-DC-5V" gate="G$1" pin="+V"/>
 <pinref part="P+6" gate="VCC" pin="VCC"/>
+<junction x="98.425" y="165.1"/>
+<junction x="98.298" y="165.1"/>
 </segment>
 <segment>
@@
 <pinref part="P+12" gate="VCC" pin="VCC"/>
 <wire x1="-82.55" y1="154.94" x2="-73.66" y2="154.94" width="0.1524" layer="91"/>
+</segment>
+<segment>
+<pinref part="U$2" gate="G$1" pin="VCC"/>
+<wire x1="-116.84" y1="162.56" x2="-113.03" y2="162.56" width="0.1524" layer="91"/>
+<wire x1="-113.03" y1="162.56" x2="-113.03" y2="119.38" width="0.1524" layer="91"/>
+<wire x1="-113.03" y1="119.38" x2="-147.32" y2="119.38" width="0.1524" layer="91"/>
+<wire x1="-147.32" y1="119.38" x2="-147.32" y2="129.54" width="0.1524" layer="91"/>
+<pinref part="JP3" gate="G$1" pin="VBUS"/>
+<wire x1="-137.16" y1="129.54" x2="-147.32" y2="129.54" width="0.2032" layer="91"/>
+<pinref part="P+15" gate="VCC" pin="VCC"/>
+<junction x="-113.03" y="119.38"/>
 </segment>
 </net>
@@
 <wire x1="-40.64" y1="1.27" x2="-40.64" y2="-10.16" width="0.1524" layer="91"/>
 <wire x1="-38.1" y1="1.27" x2="-40.64" y2="1.27" width="0.1524" layer="91"/>
+<junction x="-40.64" y="1.27"/>
 </segment>
 </net>
@@
 <wire x1="-58.42" y1="77.47" x2="-58.42" y2="81.28" width="0.1524" layer="91"/>
 <pinref part="X77" gate="-3" pin="S"/>
+<junction x="-58.42" y="81.28"/>
 </segment>
 </net>
@@
 </segment>
 </net>
-<net name="N$19" class="5">
+<net name="N$29" class="5">
 <segment>
 <pinref part="K4" gate="G$1" pin="DS1"/>
@@
 </segment>
 </net>
-<net name="N$35" class="5">
+<net name="N$25" class="5">
 <segment>
 <pinref part="K2" gate="G$1" pin="DS1"/>
@@
 </segment>
 </net>
-<net name="N$41" class="5">
+<net name="N$35" class="5">
 <segment>
 <pinref part="K6" gate="G$1" pin="DS1"/>
@@
 </segment>
 </net>
-<net name="N$40" class="5">
+<net name="N$38" class="5">
 <segment>
 <pinref part="K5" gate="G$1" pin="DS1"/>
@@
 <label x="-52.07" y="83.82" size="1.27" layer="95" rot="R180" xref="yes"/>
 </segment>
-<segment>
-<pinref part="IC2" gate="G$1" pin="VCC2"/>
-<pinref part="X11" gate="-2" pin="S"/>
-<wire x1="-73.66" y1="119.38" x2="-83.82" y2="119.38" width="0.2032" layer="91"/>
-</segment>
-</net>
-<net name="+5V" class="1">
-<segment>
-<pinref part="U$2" gate="G$1" pin="VCC"/>
-<wire x1="-116.84" y1="162.56" x2="-113.03" y2="162.56" width="0.1524" layer="91"/>
-<wire x1="-113.03" y1="162.56" x2="-113.03" y2="119.38" width="0.1524" layer="91"/>
-<wire x1="-113.03" y1="119.38" x2="-147.32" y2="119.38" width="0.1524" layer="91"/>
-<wire x1="-147.32" y1="119.38" x2="-147.32" y2="129.54" width="0.1524" layer="91"/>
-<pinref part="+3V9" gate="1" pin="+5V"/>
-<pinref part="JP3" gate="G$1" pin="VBUS"/>
-<wire x1="-137.16" y1="129.54" x2="-147.32" y2="129.54" width="0.2032" layer="91"/>
-</segment>
 </net>
 <net name="N$7" class="0">
@@
 </segment>
 </net>
+<net name="N$19" class="0">
+<segment>
+<pinref part="X11" gate="-2" pin="S"/>
+<wire x1="-83.82" y1="119.38" x2="-73.66" y2="119.38" width="0.2032" layer="91"/>
+<wire x1="-73.66" y1="119.38" x2="-73.66" y2="119.253" width="0.2032" layer="91"/>
+<junction x="-83.82" y="119.38"/>
+<pinref part="IC2" gate="G$1" pin="VCC2"/>
+<junction x="-73.66" y="119.38"/>
+</segment>
+</net>
 </nets>
 </sheet>
 </sheets>
+<errors>
+</errors>
 </schematic>
 </drawing>

Commit message: TRASAvimas
Connections:
- removed net N$15: DIODE2.C, T2.C, X77-3.S
- net +12V: now also DIODE2.C, T2.C, X77-3.S
Changed lines of the file:
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@@
 <setting verticaltext="up"/>
 </settings>
-<grid distance="0.127" unitdist="mm" unit="mm" style="lines" multiple="1" display="no" altdistance="0.01" altunitdist="inch" altunit="inch"/>
+<grid distance="0.1" unitdist="inch" unit="inch" style="lines" multiple="1" display="no" altdistance="0.01" altunitdist="inch" altunit="inch"/>
 <layers>
 <layer number="1" name="Top" color="4" fill="1" visible="no" active="no"/>
@@
 </segment>
 </net>
-<net name="N$15" class="0">
-<segment>
-<pinref part="T2" gate="1" pin="C"/>
-<wire x1="-73.66" y1="81.28" x2="-58.42" y2="81.28" width="0.1524" layer="91"/>
-<wire x1="-58.42" y1="81.28" x2="-49.53" y2="81.28" width="0.1524" layer="91"/>
-<pinref part="DIODE2" gate="1" pin="C"/>
-<wire x1="-58.42" y1="77.47" x2="-58.42" y2="81.28" width="0.1524" layer="91"/>
-<pinref part="X77" gate="-3" pin="S"/>
-<junction x="-58.42" y="81.28"/>
-</segment>
-</net>
 <net name="N$20" class="0">
 <segment>
@@
 <segment>
 <pinref part="X77" gate="-4" pin="S"/>
-<wire x1="-49.53" y1="83.82" x2="-52.07" y2="83.82" width="0.2032" layer="91"/>
+<wire x1="-49.53" y1="83.82" x2="-50.8" y2="83.82" width="0.2032" layer="91"/>
 <label x="-52.07" y="83.82" size="1.27" layer="95" rot="R180" xref="yes"/>
-</segment>
-</net>
+<pinref part="T2" gate="1" pin="C"/>
+<wire x1="-50.8" y1="83.82" x2="-52.07" y2="83.82" width="0.2032" layer="91"/>
+<wire x1="-73.66" y1="81.28" x2="-58.42" y2="81.28" width="0.1524" layer="91"/>
+<wire x1="-58.42" y1="81.28" x2="-50.8" y2="81.28" width="0.1524" layer="91"/>
+<pinref part="DIODE2" gate="1" pin="C"/>
+<wire x1="-50.8" y1="81.28" x2="-49.53" y2="81.28" width="0.1524" layer="91"/>
+<wire x1="-58.42" y1="77.47" x2="-58.42" y2="81.28" width="0.1524" layer="91"/>
+<pinref part="X77" gate="-3" pin="S"/>
+<junction x="-58.42" y="81.28"/>
+<wire x1="-50.8" y1="83.82" x2="-50.8" y2="81.28" width="0.2032" layer="91"/>
+</segment>
+</net>
