File: 3K_valdiklis_v1/3K_valdiklis_v1.2x.brd (EAGLE design)
At the start: 150 x 90 mm, 61 parts, among them IC2 L293D, IC4 ATMEGA1284, J4 HEAD3X2, K1 S202T02, K2 S202T02, K3 S202T02, K4 S202T02, K5 S202T02, K6 S202T02, T2 TIP120V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

Commit message: trasavimas
Parts:
- removed DIODE1: BAT85, SteveMarple:DIODE-TH-0.4
- added JP11, JP12, JP5, JP7, JP8, JP9: M01PTH, SparkFun-Connectors-1:1X01
- moved C7 129.4 mm to (134.0, 36.2)
- moved C6 107.6 mm to (111.1, 6.99), turned to 0 degrees
- moved C2 54.8 mm to (55.9, 34.9), turned to 0 degrees
- moved R15 39.7 mm to (68.1, 8.00)
- moved X10 34.9 mm to (61.7, 3.30)
- moved R7 25.0 mm to (87.0, 1.91), turned to 0 degrees
- moved S1 19.0 mm to (76.2, 5.08), turned to 90 degrees
- moved R10 12.1 mm to (25.4, 48.9)
- moved U$4 12.1 mm to (26.0, 9.02)
- moved JP2 10.2 mm to (12.8, 7.11)
- moved LED2 8.47 mm to (16.5, 50.2)
- moved AC-DC-5V 7.65 mm to (27.9, 12.7)
- moved C13 6.48 mm to (11.4, 48.3), turned to 90 degrees
- moved L1 6.25 mm to (40.6, 40.6), turned to 180 degrees
- moved U$3 5.24 mm to (128.3, 15.9)
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Connections:
- net !RESET: no longer DIODE1.A
- net D0: no longer R1.1
- net D1: now also R1.1; no longer R2.1
- net D10(RX1): now also IC2.2
- net D11(TX1): now also IC2.15; no longer IC2.10
- net D12: now also IC2.10; no longer IC2.2
- net D14: now also R15.2, X10.2; no longer IC2.15
- net D2: now also R2.1; no longer R3.1
- net D3: now also R3.1; no longer R4.1
- net D4: now also R4.1; no longer R5.1
- net D5(MOSI): now also R5.1; no longer R6.1
- net D6(MISO): now also R6.1; no longer R15.2, X10.2
- net MV1.1: now also X7.2; no longer X7.1
- net MV1.2: now also X7.1; no longer X7.2
- net N$18: now also JP9.1
- net N$25: now also JP11.1
- net N$29: now also JP8.1
- net N$32: now also JP12.1
- net N$35: now also JP5.1
- net N$38: now also JP7.1
- net VCC: no longer DIODE1.C
Routing:
- net D12: track 95.7 -> 26.7 mm, vias 0 -> 1
- net N$5: track 0.00 -> 63.8 mm, vias 1 -> 0
- net N$17: track 0.00 -> 63.8 mm
- net D17(SDA): track 97.5 -> 37.5 mm
- net D10(RX1): track 0.00 -> 49.8 mm
- net D16(SCL): track 73.0 -> 43.3 mm, vias 0 -> 1
- net N$20: track 27.9 -> 0.00 mm
- net !RESET: track 136.2 -> 113.1 mm
- net D14: track 36.2 -> 18.6 mm
- net D0: track 26.4 -> 9.85 mm
- net GND: track 437.2 -> 450.1 mm, vias 0 -> 1
- net D2: track 39.8 -> 28.1 mm
- net D3: track 48.5 -> 36.8 mm
- net D4: track 56.9 -> 45.4 mm
- net D1: track 31.1 -> 19.8 mm
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Other:
- board size 150 x 90 mm -> 138 x 90 mm
- board text added: "SauleVire.lt"
